File: KiCad/FujiNet_Z80Bus_Reference/SPIBUS.sch (KiCad schematic (older format))
At the start: 13 parts, among them IC10 74595N, IC11 74165N, IC12 74165N, IC17 74165N, IC18 74165N, IC3 74595N, IC8 74595N, IC9 74595N

Commit message: Last KiCad5 commit
Parts:
- added J2: DIAG-ESP_SPI, Connector_PinHeader_2.54mm:PinHeader_1x08_P2.54mm_Vertical, symbol Connector:Conn_01x08_Female
- added J3: DIAG-Z80_CONTROL, Connector_PinHeader_2.54mm:PinHeader_1x08_P2.54mm_Vertical, symbol Connector:Conn_01x08_Female
- added J4: DIAG-ESP_CONTROL, Connector_PinHeader_2.54mm:PinHeader_1x08_P2.54mm_Vertical, symbol Connector:Conn_01x08_Female
- added J5: DIAG-LOCAL_ADD_HIGH, Connector_PinHeader_2.54mm:PinHeader_1x08_P2.54mm_Vertical, symbol Connector:Conn_01x08_Female
- added J6: DIAG-LOCAL_ADD_LOW, Connector_PinHeader_2.54mm:PinHeader_1x08_P2.54mm_Vertical, symbol Connector:Conn_01x08_Female
- added J7: DIAG-LOCAL_DATA, Connector_PinHeader_2.54mm:PinHeader_1x08_P2.54mm_Vertical, symbol Connector:Conn_01x08_Female
Connections:
- net ESP_CONTROL_BUSRQ: now also J4.5 (Pin_5)
- net ESP_CONTROL_IORQ: now also J4.3 (Pin_3)
- net ESP_CONTROL_MEMRQ: now also J4.4 (Pin_4)
- net ESP_CONTROL_NMI: now also J4.8 (Pin_8)
- net ESP_CONTROL_RD: now also J4.1 (Pin_1)
- net ESP_CONTROL_ROMCS: now also J4.7 (Pin_7)
- net ESP_CONTROL_WAIT: now also J4.6 (Pin_6)
- net ESP_CONTROL_WR: now also J2.4 (Pin_4), J4.2 (Pin_2)
- net ESP_SPI.CE: now also J2.7 (Pin_7)
- net ESP_SPI.MISO: now also J2.2 (Pin_2)
- net ESP_SPI.MOSI: now also J2.1 (Pin_1)
- net ESP_SPI.OE: now also J2.5 (Pin_5)
- net ESP_SPI.PL: now also J2.8 (Pin_8)
- net ESP_SPI.SCK: now also J2.6 (Pin_6)
- net ESP_SPI.STC: now also J2.3 (Pin_3)
- net LOCAL_ADD_0: now also J6.1 (Pin_1)
- net LOCAL_ADD_1: now also J6.2 (Pin_2)
- net LOCAL_ADD_10: now also J5.3 (Pin_3)
- net LOCAL_ADD_11: now also J5.4 (Pin_4)
- net LOCAL_ADD_12: now also J5.5 (Pin_5)
- net LOCAL_ADD_13: now also J5.6 (Pin_6)
- net LOCAL_ADD_14: now also J5.7 (Pin_7)
- net LOCAL_ADD_15: now also J5.8 (Pin_8)
- net LOCAL_ADD_2: now also J6.3 (Pin_3)
- net LOCAL_ADD_3: now also J6.4 (Pin_4)
- net LOCAL_ADD_4: now also J6.5 (Pin_5)
- net LOCAL_ADD_5: now also J6.6 (Pin_6)
- net LOCAL_ADD_6: now also J6.7 (Pin_7)
- net LOCAL_ADD_7: now also J6.8 (Pin_8)
- net LOCAL_ADD_8: now also J5.1 (Pin_1)
- net LOCAL_ADD_9: now also J5.2 (Pin_2)
- net LOCAL_DATA_0: now also J7.1 (Pin_1)
- net LOCAL_DATA_1: now also J7.2 (Pin_2)
- net LOCAL_DATA_2: now also J7.3 (Pin_3)
- net LOCAL_DATA_3: now also J7.4 (Pin_4)
- net LOCAL_DATA_4: now also J7.5 (Pin_5)
- net LOCAL_DATA_5: now also J7.6 (Pin_6)
- net LOCAL_DATA_6: now also J7.7 (Pin_7)
- net LOCAL_DATA_7: now also J7.8 (Pin_8)
- net Z80_BUSACK: now also J3.7 (Pin_7)
- net Z80_BUSRQ: now also J3.5 (Pin_5)
- net Z80_IORQ: now also J3.3 (Pin_3)
- net Z80_MEMRQ: now also J3.4 (Pin_4)
- net Z80_NMI: now also J3.8 (Pin_8)
- net Z80_RD: now also J3.1 (Pin_1)
- net Z80_WAIT: now also J3.6 (Pin_6)
- net Z80_WR: now also J3.2 (Pin_2)
