File: KiCad7/FujiNet_Z80Bus_ReferenceDesign/Logic core/Z80 BUS CONTROL.kicad_sch (KiCad schematic)
At the start: 9 parts, among them IC6 74HC32N, IC7 74HC32N

Commit message: KiCAD PCB layout testing
Parts:
- R12, R13: footprint (none) -> Resistor_THT:R_Axial_DIN0207_L6.3mm_D2.5mm_P10.16mm_Horizontal
Changed lines of the file:
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@@
       (effects (font (size 1.27 1.27)))
     )
-    (property "Footprint" "" (at 86.36 137.668 90)
+    (property "Footprint" "Resistor_THT:R_Axial_DIN0207_L6.3mm_D2.5mm_P10.16mm_Horizontal" (at 86.36 137.668 90)
       (effects (font (size 1.27 1.27)) hide)
     )
@@
       (effects (font (size 1.27 1.27)))
     )
-    (property "Footprint" "" (at 86.36 66.802 90)
+    (property "Footprint" "Resistor_THT:R_Axial_DIN0207_L6.3mm_D2.5mm_P10.16mm_Horizontal" (at 86.36 66.802 90)
       (effects (font (size 1.27 1.27)) hide)
     )
