File: KiCad7/FujiNet_Z80Bus_ReferenceDesign/FujiNet_Z80Bus_ReferenceDesign.kicad_pcb (KiCad board)
At the start: 2 copper layers, 180.3 x 119.4 mm, 76 parts, among them IC13 7432N, IC15 7408N, IC19 7432N, IC2 7404N, IC20 7408N, IC21 7432N, IC22 7432N, IC3 7474N, IC4 7432N, IC5 7408N, IC6 74590N, IC7 74590N, J2 DIAG-ESP_SPI, J3 DIAG-Z80_CONTROL, J4 DIAG-ESP_CONTROL, J5 DIAG-LOCAL_ADD_HIGH, J6 DIAG-LOCAL_ADD_LOW, J7 DIAG-LOCAL_DATA, J8 DIAG-HOST_SYSTEM_BUS, Q1 2N2222 (BC337), U1 FREENOVE_ESP32-WROVER-DEV

Commit message: KiCAD attempt to route a single board (failed)
Parts:
- removed IC13, IC19, IC21, IC22: 7432N, Package_DIP:DIP-14_W7.62mm_Socket
- removed IC15, IC20: 7408N, Package_DIP:DIP-14_W7.62mm_Socket
- removed J2: DIAG-ESP_SPI, Connector_PinHeader_2.54mm:PinHeader_1x08_P2.54mm_Vertical
- removed J3: DIAG-Z80_CONTROL, Connector_PinHeader_2.54mm:PinHeader_1x08_P2.54mm_Vertical
- removed J4: DIAG-ESP_CONTROL, Connector_PinHeader_2.54mm:PinHeader_1x08_P2.54mm_Vertical
- removed J5: DIAG-LOCAL_ADD_HIGH, Connector_PinHeader_2.54mm:PinHeader_1x08_P2.54mm_Vertical
- removed J6: DIAG-LOCAL_ADD_LOW, Connector_PinHeader_2.54mm:PinHeader_1x08_P2.54mm_Vertical
- removed J7: DIAG-LOCAL_DATA, Connector_PinHeader_2.54mm:PinHeader_1x08_P2.54mm_Vertical
- removed JP4: PINHD-POWER/RESET, Connector_PinSocket_2.54mm:PinSocket_1x03_P2.54mm_Vertical
- removed RN4: 4609M-101-103LF, Resistor_THT:R_Array_SIP9
- added IC1: 7432N, Package_DIP:DIP-14_W7.62mm_Socket, F.Cu at (34.2, 115.0)
- added IC10: 7408N, Package_DIP:DIP-14_W7.62mm_Socket, F.Cu at (64.9, 114.7)
- added IC11: 74590N, Package_DIP:DIP-16_W7.62mm_Socket, F.Cu at (110.3, 76.9)
- added IC12: 74590N, Package_DIP:DIP-16_W7.62mm_Socket, F.Cu at (116.1, 55.4)
- added IC8: 7432N, Package_DIP:DIP-14_W7.62mm_Socket, F.Cu at (65.4, 42.5)
- added IC9: 7408N, Package_DIP:DIP-14_W7.62mm_Socket, F.Cu at (65.1, 60.0)
- added JP2: PINHD-POWER/RESET, Connector_PinSocket_2.54mm:PinSocket_1x03_P2.54mm_Vertical, F.Cu at (43.4, 173.4)
- added RN1: 4609M-101-103LF, Resistor_THT:R_Array_SIP9, F.Cu at (197.2, 51.1)
- C1: value 10UF -> 10 uf
- C2: value 10UF -> .1 uf
- C3: value 10 uf -> .1 uf
- C4, C5: value .1 uf -> 10UF
- IC4: value 7432N -> 7408N
- IC5: value 7408N -> 7432N
- IC6, IC7: value 74590N -> 7432N; footprint Package_DIP:DIP-16_W7.62mm_Socket -> Package_DIP:DIP-14_W7.62mm_Socket
- R2: value 1K -> 22K
- R6: value 22K -> 10K
- R7: value 1K -> 10K
- R8, R9: value 10K -> 1K
- SPI-LOCAL_DATA.IN1: moved to F.Cu
- moved C5 194.3 mm to (28.8, 60.0)
- moved R2 193.7 mm to (28.8, 42.0), turned to -90 degrees
- moved D7 188.2 mm to (218.1, 38.5), turned to 0 degrees
- moved IC4 181.5 mm to (34.1, 60.0), turned to 90 degrees
- moved C4 181.0 mm to (28.8, 73.0)
- moved D8 179.4 mm to (218.1, 49.0), turned to 0 degrees
- moved D9 179.1 mm to (218.1, 44.4), turned to 0 degrees
- moved D4 162.2 mm to (51.7, 129.5), turned to 90 degrees
- moved D6 148.0 mm to (64.8, 134.5), turned to -90 degrees
- moved R4 144.9 mm to (223.3, 33.2), turned to 0 degrees
- moved C1 144.9 mm to (52.2, 178.8)
- moved C3 143.0 mm to (63.0, 178.9), turned to 90 degrees
- moved ESP_CONTROL_DIRECTOR1 139.2 mm to (33.7, 154.3), turned to 90 degrees
- moved C2 138.4 mm to (73.8, 178.9), turned to 90 degrees
- moved D12 134.7 mm to (74.3, 134.6), turned to -90 degrees
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Connections:
- C1 pad 1: /CORE/ESP_WAIT_RESET -> +5V
- C2 pad 1: Net-(IC5A-I0) -> +5V
- C4 pad 1: +5V -> /CORE/ESP_WAIT_RESET
- C5 pad 1: +5V -> Net-(IC4A-I0)
- D10 pad 1: /CORE/ESP_CONTROL.NMI -> Net-(D10-K)
- D10 pad 2: /CORE/Z80_CONTROL.NMI -> +5V
- D11 pad 1: /Z80_HARDLOCK_RESET -> Net-(D11-K)
- D11 pad 2: /CORE/ESP_INT -> +5V
- D12 pad 1: /CORE/Z80_CONTROL.BUSACK -> /CORE/ESP_CONTROL.BUSRQ
- D12 pad 2: /CORE/ESP_INT -> /CORE/Z80_CONTROL.BUSRQ
- D13 pad 1: Net-(D13-K) -> /CORE/ESP_CONTROL.WAIT
- D14 pad 1: Net-(D14-K) -> /CORE/ESP_CONTROL.ROMCS
- D14 pad 2: +5V -> /CORE/Z80_CONTROL.ROMCS
- D15 pad 1: Net-(D15-K) -> /CORE/ESP_CONTROL.NMI
- D15 pad 2: +5V -> /CORE/Z80_CONTROL.NMI
- D2 pad 1: /CORE/ESP_CONTROL.BUSRQ -> Net-(D2-K)
- D2 pad 2: /CORE/Z80_ADD_CONNECT -> /CORE/Z80_CONTROL.RESET
- D3 pad 2: /CORE/Z80_DATA_CONNECT -> /CORE/Z80_ADD_CONNECT
- D4 pad 1: Net-(D4-K) -> /CORE/ESP_CONTROL.BUSRQ
- D4 pad 2: /CORE/Z80_CONTROL.RESET -> /CORE/Z80_DATA_CONNECT
- D6 pad 1: /CORE/Z80_CONTROL.WAIT -> Net-(D6-K)
- D6 pad 2: /CORE/ESP_INT -> /CORE/Z80_CONTROL.WAIT
- D7 pad 1: /CORE/ESP_CONTROL.BUSRQ -> /CORE/Z80_CONTROL.WAIT
- D7 pad 2: /CORE/Z80_CONTROL.BUSRQ -> /CORE/ESP_INT
- D8 pad 1: /CORE/ESP_CONTROL.WAIT -> /Z80_HARDLOCK_RESET
- D8 pad 2: /CORE/Z80_CONTROL.WAIT -> /CORE/ESP_INT
- D9 pad 1: /CORE/ESP_CONTROL.ROMCS -> /CORE/Z80_CONTROL.BUSACK
- D9 pad 2: /CORE/Z80_CONTROL.ROMCS -> /CORE/ESP_INT
- ESP_CONTROL_BIAS1 pad 1: Net-(D16-K) -> Net-(D11-K)
- IC2 pad 10: Net-(IC2E-O) -> Net-(IC1C-I0)
- IC3 pad 8: Net-(D13-K) -> Net-(D6-K)
- IC4 pad 1: (no net) -> Net-(IC4A-I0)
- IC4 pad 10: /CORE/ESP_CONTROL.BUSRQ -> (no net)
- IC4 pad 2: (no net) -> Net-(IC2C-O)
- IC4 pad 3: (no net) -> /CORE/CLR_Z80_HARDLOCK
- IC4 pad 4: (no net) -> /CORE/ESP_CONTROL.MEMRQ
- IC4 pad 5: (no net) -> /CORE/ESP_CONTROL.IORQ
- IC4 pad 6: (no net) -> Net-(IC2E-I)
- IC4 pad 8: /ESP_IOD_CONFIG -> (no net)
- IC4 pad 9: Net-(IC2E-O) -> (no net)
- IC5 pad 1: Net-(IC5A-I0) -> (no net)
- IC5 pad 10: (no net) -> /CORE/Z80_CONTROL.IORQ
- IC5 pad 2: Net-(IC2C-O) -> (no net)
- IC5 pad 3: /CORE/CLR_Z80_HARDLOCK -> (no net)
- IC5 pad 4: /CORE/ESP_CONTROL.MEMRQ -> (no net)
- IC5 pad 5: /CORE/ESP_CONTROL.IORQ -> (no net)
- IC5 pad 6: Net-(IC2E-I) -> (no net)
- IC5 pad 8: (no net) -> Net-(IC5C-O)
- IC5 pad 9: (no net) -> /CORE/ESP_HARDLOCK
- IC6 pad 1: /CACHE/LOCAL_A1 -> /PERM_Z80_IORQ
- IC6 pad 10: /Z80_HARDLOCK -> /CORE/Z80_DATA_CONNECT
- IC6 pad 11: /CACHE/CACHE_DATASTATUS+PERM_Z80_IORQ -> /PERM_Z80_IORQ
- IC6 pad 12: /CACHE_DATASTATUS -> /CORE/IORQ_FILTER_BIT
- IC6 pad 13: /CACHE/CACHE_DATASTATUS+PERM_Z80_IORQ -> Net-(IC5C-O)
- IC6 pad 14: /CACHE_DATASTATUS -> (no net)
- IC6 pad 2: /CACHE/LOCAL_A2 -> /!CACHE_DATASTATUS
- IC6 pad 3: /CACHE/LOCAL_A3 -> Net-(IC6A-O)
- IC6 pad 4: /CACHE/LOCAL_A4 -> /CORE/Z80_CONTROL.RD
- IC6 pad 5: /CACHE/LOCAL_A5 -> /PERM_Z80_IORQ
- IC6 pad 6: /CACHE/LOCAL_A6 -> Net-(IC6B-O)
- IC6 pad 7: /CACHE/LOCAL_A7 -> (no net)
- IC6 pad 8: (no net) -> Net-(IC6C-O)
- IC6 pad 9: Net-(IC6A-RCO) -> /CORE/ESP_CONTROL.WR
- IC7 pad 1: /CACHE/LOCAL_A9 -> /CORE/Z80_ADD_CONNECT
- IC7 pad 10: /Z80_HARDLOCK -> Net-(IC6C-O)
- IC7 pad 11: Net-(IC6A-RCO) -> /Z80 BUS/Z80_DATA_OE
- IC7 pad 12: /CACHE_DATASTATUS -> /CORE/Z80_DATA_CONNECT
- IC7 pad 13: Net-(IC6A-RCO) -> /PERM_Z80_IORQ
- IC7 pad 14: /CACHE_DATASTATUS -> (no net)
- IC7 pad 2: /CACHE/LOCAL_A10 -> Net-(IC6A-O)
- IC7 pad 3: /CACHE/LOCAL_A11 -> /Z80 BUS/Z80_ADD_OE
- IC7 pad 4: unconnected-(IC7A-QE-Pad4) -> /ESP_IOD_CONFIG
- IC7 pad 5: unconnected-(IC7A-QF-Pad5) -> /CORE/ESP_CONTROL.MEMRQ
- IC7 pad 6: unconnected-(IC7A-QG-Pad6) -> /Z80 BUS/Z80_ADD_DIR
- IC7 pad 7: unconnected-(IC7A-QH-Pad7) -> (no net)
- IC7 pad 8: (no net) -> /Z80 BUS/Z80_DATA_DIR
- IC7 pad 9: unconnected-(IC7A-RCO-Pad9) -> Net-(IC6B-O)
- J8 pad 12: /RIO/Z80_D0 -> /RIO/Z80_A0
- J8 pad 13: /RIO/Z80_D1 -> /RIO/Z80_A1
- J8 pad 14: /RIO/Z80_D2 -> /RIO/Z80_A2
- J8 pad 15: /RIO/Z80_D3 -> /RIO/Z80_A3
- J8 pad 16: /RIO/Z80_D4 -> /RIO/Z80_A4
- J8 pad 17: /RIO/Z80_D5 -> /RIO/Z80_A5
- J8 pad 18: /RIO/Z80_D6 -> /RIO/Z80_A6
- J8 pad 19: /RIO/Z80_D7 -> /RIO/Z80_A7
- J8 pad 20: /RIO/Z80_A0 -> /RIO/Z80_A8
- J8 pad 21: /RIO/Z80_A1 -> /RIO/Z80_A9
- J8 pad 22: /RIO/Z80_A2 -> /RIO/Z80_A10
- J8 pad 23: /RIO/Z80_A3 -> /RIO/Z80_A11
- J8 pad 24: /RIO/Z80_A4 -> /RIO/Z80_A12
- J8 pad 25: /RIO/Z80_A5 -> /RIO/Z80_A13
- J8 pad 26: /RIO/Z80_A6 -> /RIO/Z80_A14
- J8 pad 27: /RIO/Z80_A7 -> /RIO/Z80_A15
- J8 pad 28: /RIO/Z80_A8 -> /RIO/Z80_D0
- J8 pad 29: /RIO/Z80_A9 -> /RIO/Z80_D1
- J8 pad 30: /RIO/Z80_A10 -> /RIO/Z80_D2
- J8 pad 31: /RIO/Z80_A11 -> /RIO/Z80_D3
- J8 pad 32: /RIO/Z80_A12 -> /RIO/Z80_D4
- J8 pad 33: /RIO/Z80_A13 -> /RIO/Z80_D5
- J8 pad 34: /RIO/Z80_A14 -> /RIO/Z80_D6
- J8 pad 35: /RIO/Z80_A15 -> /RIO/Z80_D7
- LOCAL_DATA_BIAS1 pad 1: Net-(D15-K) -> Net-(D10-K)
- R10 pad 1: /CACHE/CACHE_CE2 -> +5V
- R10 pad 2: +5V -> /RIO/RIO_CE2
- R11 pad 1: +5V -> /CACHE/CACHE_CE2
- R11 pad 2: /RIO/RIO_CE2 -> +5V
- R2 pad 1: /CACHE_DATASTATUS -> +5V
- R2 pad 2: Net-(Q1-B) -> Net-(IC4A-I0)
- R4 pad 1: +5V -> /CORE/ESP_INT
- R4 pad 2: Net-(IC5A-I0) -> GND
- R5 pad 1: /CORE/ESP_INT -> +5V
- R5 pad 2: GND -> /CORE/ESP_SPI_INT.MR
- R6 pad 1: +5V -> /CACHE_DATASTATUS
- R6 pad 2: /CORE/ESP_SPI_INT.MR -> +5V
- R7 pad 1: /!CACHE_DATASTATUS -> Net-(RIO_DECODER1A-DIR)
- R8 pad 1: Net-(RIO_DECODER1A-DIR) -> /!CACHE_DATASTATUS
- R9 pad 2: +5V -> Net-(Q1-B)
- U1 pad 35: Net-(D4-K) -> Net-(D2-K)
Other:
- board size 180.3 x 119.4 mm -> 239.3 x 158.4 mm

Commit message: KiCad massive refactoring to enable modular PCB design
Parts:
- removed C4, C5: 10UF, Capacitor_THT:CP_Radial_D8.0mm_P5.00mm
- removed D16, D3, D4, D6: 1N4148, Diode_THT:D_T-1_P5.08mm_Horizontal
- removed IC10, IC4, IC9: 7408N, Package_DIP:DIP-14_W7.62mm_Socket
- removed IC2: 7404N, Package_DIP:DIP-14_W7.62mm_Socket
- removed IC3: 7474N, Package_DIP:DIP-14_W7.62mm_Socket
- removed IC5, IC6, IC7, IC8: 7432N, Package_DIP:DIP-14_W7.62mm_Socket
- removed Q1: 2N2222 (BC337), Package_TO_SOT_THT:TO-92
- removed R2: 22K, Resistor_THT:R_Axial_DIN0207_L6.3mm_D2.5mm_P10.16mm_Horizontal
- removed R9: 1K, Resistor_THT:R_Axial_DIN0207_L6.3mm_D2.5mm_P10.16mm_Horizontal
- removed RIO_CONTROL1: 74244N, Package_DIP:DIP-20_W7.62mm_Socket
- removed RN1: 4609M-101-103LF, Resistor_THT:R_Array_SIP9
- added J10: Logic core connector (main), Connector_PinHeader_2.54mm:PinHeader_2x40_P2.54mm_Vertical, F.Cu at (245.5, 163.6)
- moved LOCAL_DATA_BIAS1 83.4 mm to (166.6, 54.4)
- moved Z80-LOCAL_DATA1 80.0 mm to (145.2, 124.6)
- moved RIO1 74.9 mm to (188.7, 85.8), turned to 0 degrees
- moved R10 74.3 mm to (207.7, 80.7), turned to -90 degrees
- moved R6 71.5 mm to (143.2, 38.0), turned to 0 degrees
- moved SPI-LOCAL_DATA.IN1 65.5 mm to (178.7, 84.9)
- moved SPI-LOCAL_DATA.OUT1 63.2 mm to (171.7, 47.9)
- moved R8 62.1 mm to (143.7, 30.9), turned to 0 degrees
- moved SPI-LOCAL_ADD_L.OUT1 50.5 mm to (80.6, 66.2)
- moved SPI-ESP_CONTROL.OUT1 50.2 mm to (50.0, 36.8)
- moved D11 50.2 mm to (49.4, 31.7)
- moved ESP_CONTROL_BIAS1 50.2 mm to (44.6, 31.7)
- moved R5 50.2 mm to (61.4, 31.5)
- moved CACHE1 50.2 mm to (141.3, 68.4), turned to 0 degrees
- moved SPI-LOCAL_ADDR_L.IN1 47.6 mm to (91.4, 101.1)
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Connections:
- net /CACHE/CACHE_DATASTATUS+PERM_Z80_IORQ renamed /CACHE_CONTROL.DATASTATUS+PERM_Z80_IORQ
- net /CACHE/LOCAL_A0 renamed /LOCAL_A0
- net /CACHE/LOCAL_A1 renamed /LOCAL_A1
- net /CACHE/LOCAL_A10 renamed /LOCAL_A10
- net /CACHE/LOCAL_A11 renamed /LOCAL_A11
- net /CACHE/LOCAL_A12 renamed /LOCAL_A12
- net /CACHE/LOCAL_A13 renamed /LOCAL_A13
- net /CACHE/LOCAL_A14 renamed /LOCAL_A14
- net /CACHE/LOCAL_A15 renamed /LOCAL_A15
- net /CACHE/LOCAL_A2 renamed /LOCAL_A2
- net /CACHE/LOCAL_A3 renamed /LOCAL_A3
- net /CACHE/LOCAL_A4 renamed /LOCAL_A4
- net /CACHE/LOCAL_A5 renamed /LOCAL_A5
- net /CACHE/LOCAL_A6 renamed /LOCAL_A6
- net /CACHE/LOCAL_A7 renamed /LOCAL_A7
- net /CACHE/LOCAL_A8 renamed /LOCAL_A8
- net /CACHE/LOCAL_A9 renamed /LOCAL_A9
- net /CACHE/LOCAL_CONTROL.IORQ renamed /LOCAL_CONTROL.IORQ
- net /CACHE/LOCAL_CONTROL.MEMRQ renamed /LOCAL_CONTROL.MEMRQ
- net /CACHE/LOCAL_CONTROL.RD renamed /LOCAL_CONTROL.RD
- net /CACHE/LOCAL_CONTROL.WR renamed /LOCAL_CONTROL.WR
- net /CACHE/LOCAL_D0 renamed /LOCAL_D0
- net /CACHE/LOCAL_D1 renamed /LOCAL_D1
- net /CACHE/LOCAL_D2 renamed /LOCAL_D2
- net /CACHE/LOCAL_D3 renamed /LOCAL_D3
- net /CACHE/LOCAL_D4 renamed /LOCAL_D4
- net /CACHE/LOCAL_D5 renamed /LOCAL_D5
- net /CACHE/LOCAL_D6 renamed /LOCAL_D6
- net /CACHE/LOCAL_D7 renamed /LOCAL_D7
- net /CORE/ESP_CONTROL.BUSRQ renamed /ESP_CONTROL.BUSRQ
- net /CORE/ESP_CONTROL.IORQ renamed /ESP_CONTROL.IORQ
- net /CORE/ESP_CONTROL.MEMRQ renamed /ESP_CONTROL.MEMRQ
- net /CORE/ESP_CONTROL.NMI renamed /ESP_CONTROL.NMI
- net /CORE/ESP_CONTROL.RD renamed /ESP_CONTROL.RD
- net /CORE/ESP_CONTROL.ROMCS renamed /ESP_CONTROL.ROMCS
- net /CORE/ESP_CONTROL.WAIT renamed /ESP_CONTROL.WAIT
- net /CORE/ESP_CONTROL.WR renamed /ESP_CONTROL.WR
- net /RIO/DEC_OE renamed /RIO_CONTROL.OE
- net /Z80 BUS/Z80_ADD_DIR renamed /Z80_BUS_CONTROL.Z80_ADD_DIR
- net /Z80 BUS/Z80_ADD_OE renamed /Z80_BUS_CONTROL.Z80_ADD_OE
- CACHE1 pad 2: /CACHE/CACHE_A16 -> /CACHE_CONTROL.A16
- CACHE1 pad 22: /CACHE/CACHE_CS -> /CACHE_CONTROL.CS
- CACHE1 pad 24: /CACHE/CACHE_OE -> /CACHE_CONTROL.OE
- CACHE1 pad 29: /CACHE/CACHE_WE -> /CACHE_CONTROL.WE
- D12 pad 2: /CORE/Z80_CONTROL.BUSRQ -> /Z80_CONTROL.BUSRQ
- D13 pad 2: /CORE/Z80_CONTROL.WAIT -> /Z80_CONTROL.WAIT
- D14 pad 2: /CORE/Z80_CONTROL.ROMCS -> /Z80_CONTROL.ROMCS
- D15 pad 2: /CORE/Z80_CONTROL.NMI -> /Z80_CONTROL.NMI
- D2 pad 2: /CORE/Z80_CONTROL.RESET -> /Z80_CONTROL.RESET
- D7 pad 1: /CORE/Z80_CONTROL.WAIT -> /Z80_CONTROL.WAIT
- D8 pad 1: /Z80_HARDLOCK_RESET -> /CORE/Z80_HARDLOCK_RESET
- D9 pad 1: /CORE/Z80_CONTROL.BUSACK -> /Z80_CONTROL.BUSACK
- ESP_CONTROL_DIRECTOR1 pad 1: /CORE/!ESP_HARDLOCK -> /ESP_HARDLOCK
- ESP_CONTROL_DIRECTOR1 pad 3: /CORE/Z80_CONTROL.MEMRQ -> /Z80_CONTROL.MEMRQ
- ESP_CONTROL_DIRECTOR1 pad 5: /CORE/Z80_CONTROL.IORQ -> /Z80_CONTROL.IORQ
- ESP_CONTROL_DIRECTOR1 pad 7: /CORE/Z80_CONTROL.WR -> /Z80_CONTROL.WR
- ESP_CONTROL_DIRECTOR1 pad 9: /CORE/Z80_CONTROL.RD -> /Z80_CONTROL.RD
- ESP_CONTROL_DIRECTOR_BIAS1 pad 6: /CORE/Z80_ADD_CONNECT -> unconnected-(ESP_CONTROL_DIRECTOR_BIAS1-Pad6)
- ESP_CONTROL_DIRECTOR_BIAS1 pad 7: /CORE/Z80_DATA_CONNECT -> unconnected-(ESP_CONTROL_DIRECTOR_BIAS1-Pad7)
- ESP_CONTROL_DIRECTOR_BIAS1 pad 8: /CORE/ESP_WAIT_RESET -> unconnected-(ESP_CONTROL_DIRECTOR_BIAS1-Pad8)
- IC1 pad 2: /CORE/ESP_HARDLOCK -> /ESP_HARDLOCK
- IC1 pad 3: /CORE/PRE_Z80_HARDLOCK -> /Logic core/PRE_Z80_HARDLOCK
- IC1 pad 8: /ESP_IOD_CONFIG -> /Logic core/ESP_IOD_CONFIG
- J8 pad 1: GND -> /Z80_CONTROL.RD
- J8 pad 10: /CORE/Z80_CONTROL.BUSACK -> /Z80_CONTROL.RESET
- J8 pad 11: /CORE/Z80_CONTROL.RESET -> /Z80_A0
- J8 pad 12: /RIO/Z80_A0 -> /Z80_A1
- J8 pad 13: /RIO/Z80_A1 -> /Z80_A2
- J8 pad 14: /RIO/Z80_A2 -> /Z80_A3
- J8 pad 15: /RIO/Z80_A3 -> /Z80_A4
- J8 pad 16: /RIO/Z80_A4 -> /Z80_A5
- J8 pad 17: /RIO/Z80_A5 -> /Z80_A6
- J8 pad 18: /RIO/Z80_A6 -> /Z80_A7
- J8 pad 19: /RIO/Z80_A7 -> /Z80_A8
- J8 pad 2: /CORE/Z80_CONTROL.RD -> /Z80_CONTROL.WR
- J8 pad 20: /RIO/Z80_A8 -> /Z80_A9
- J8 pad 21: /RIO/Z80_A9 -> /Z80_A10
- J8 pad 22: /RIO/Z80_A10 -> /Z80_A11
- J8 pad 23: /RIO/Z80_A11 -> /Z80_A12
- J8 pad 24: /RIO/Z80_A12 -> /Z80_A13
- J8 pad 25: /RIO/Z80_A13 -> /Z80_A14
- J8 pad 26: /RIO/Z80_A14 -> /Z80_A15
- J8 pad 27: /RIO/Z80_A15 -> /Z80_D0
- J8 pad 28: /RIO/Z80_D0 -> /Z80_D1
- J8 pad 29: /RIO/Z80_D1 -> /Z80_D2
- J8 pad 3: /CORE/Z80_CONTROL.WR -> /Z80_CONTROL.IORQ
- J8 pad 30: /RIO/Z80_D2 -> /Z80_D3
- J8 pad 31: /RIO/Z80_D3 -> /Z80_D4
- J8 pad 32: /RIO/Z80_D4 -> /Z80_D5
- J8 pad 33: /RIO/Z80_D5 -> /Z80_D6
- J8 pad 34: /RIO/Z80_D6 -> /Z80_D7
- J8 pad 35: /RIO/Z80_D7 -> unconnected-(J8-Pin_35-Pad35)
- J8 pad 39: unconnected-(J8-Pin_39-Pad39) -> /Z80 BUS/VCC
- J8 pad 4: /CORE/Z80_CONTROL.IORQ -> /Z80_CONTROL.MEMRQ
- J8 pad 40: /Z80 BUS/VCC -> GND
- J8 pad 5: /CORE/Z80_CONTROL.MEMRQ -> /Z80_CONTROL.BUSRQ
- J8 pad 6: /CORE/Z80_CONTROL.BUSRQ -> /Z80_CONTROL.WAIT
- J8 pad 7: /CORE/Z80_CONTROL.WAIT -> /Z80_CONTROL.NMI
- J8 pad 8: /CORE/Z80_CONTROL.NMI -> /Z80_CONTROL.ROMCS
- J8 pad 9: /CORE/Z80_CONTROL.ROMCS -> /Z80_CONTROL.BUSACK
- JP1 pad 2: /CORE/IORQ_FILTER_BIT -> /IORQ_FILTER_BIT
- JP1 pad 3: /RIO/Z80_A0 -> /Z80_A0
- JP2 pad 1: /CORE/Z80_CONTROL.RESET -> /Z80_CONTROL.RESET
- RIO1 pad 10: /RIO/Z80_A2 -> /Z80_A2
- RIO1 pad 11: /RIO/Z80_A1 -> /Z80_A1
- RIO1 pad 12: /RIO/Z80_A0 -> /Z80_A0
- RIO1 pad 2: /RIO/DEC16 -> /RIO_CONTROL.A16
- RIO1 pad 22: /RIO/DEC_CE -> /RIO_CONTROL.CE
- RIO1 pad 23: /RIO/Z80_A10 -> /Z80_A10
- RIO1 pad 25: /RIO/Z80_A11 -> /Z80_A11
- RIO1 pad 26: /RIO/Z80_A9 -> /Z80_A9
- RIO1 pad 27: /RIO/Z80_A8 -> /Z80_A8
- RIO1 pad 28: /RIO/Z80_A13 -> /Z80_A13
- RIO1 pad 29: /RIO/DEC_WE -> /RIO/RIO_CONTROL.WE
- RIO1 pad 3: /RIO/DEC14 -> /RIO_CONTROL.A14
- RIO1 pad 31: /RIO/DEC15 -> /RIO_CONTROL.A15
- RIO1 pad 4: /RIO/Z80_A12 -> /Z80_A12
- RIO1 pad 5: /RIO/Z80_A7 -> /Z80_A7
- RIO1 pad 6: /RIO/Z80_A6 -> /Z80_A6
- RIO1 pad 7: /RIO/Z80_A5 -> /Z80_A5
- RIO1 pad 8: /RIO/Z80_A4 -> /Z80_A4
- RIO1 pad 9: /RIO/Z80_A3 -> /Z80_A3
- SPI-Z80_CONTROL.IN1 pad 11: /CORE/Z80_CONTROL.RD -> /Z80_CONTROL.RD
- SPI-Z80_CONTROL.IN1 pad 12: /CORE/Z80_CONTROL.WR -> /Z80_CONTROL.WR
- SPI-Z80_CONTROL.IN1 pad 13: /CORE/Z80_CONTROL.IORQ -> /Z80_CONTROL.IORQ
- SPI-Z80_CONTROL.IN1 pad 14: /CORE/Z80_CONTROL.MEMRQ -> /Z80_CONTROL.MEMRQ
- SPI-Z80_CONTROL.IN1 pad 3: /CORE/Z80_CONTROL.BUSRQ -> /Z80_CONTROL.BUSRQ
- SPI-Z80_CONTROL.IN1 pad 4: /CORE/Z80_CONTROL.WAIT -> /Z80_CONTROL.WAIT
- SPI-Z80_CONTROL.IN1 pad 5: /CORE/Z80_CONTROL.BUSACK -> /Z80_CONTROL.BUSACK
- SPI-Z80_CONTROL.IN1 pad 6: /CORE/Z80_CONTROL.NMI -> /Z80_CONTROL.NMI
- U1 pad 18: /CORE/ESP_WAIT_RESET -> /ESP_WAIT_RESET
- U1 pad 26: /CORE/ESP_HARDLOCK -> /!ESP_HARDLOCK
- Z80-LOCAL_DATA1 pad 1: /Z80 BUS/Z80_DATA_DIR -> /Z80_BUS_CONTROL.Z80_DATA_DIR
- Z80-LOCAL_DATA1 pad 19: /Z80 BUS/Z80_DATA_OE -> /Z80_BUS_CONTROL.Z80_DATA_OE
- Z80-LOCAL_DATA1 pad 2: /RIO/Z80_D0 -> /Z80_D0
- Z80-LOCAL_DATA1 pad 3: /RIO/Z80_D1 -> /Z80_D1
- Z80-LOCAL_DATA1 pad 4: /RIO/Z80_D2 -> /Z80_D2
- Z80-LOCAL_DATA1 pad 5: /RIO/Z80_D3 -> /Z80_D3
- Z80-LOCAL_DATA1 pad 6: /RIO/Z80_D4 -> /Z80_D4
- Z80-LOCAL_DATA1 pad 7: /RIO/Z80_D5 -> /Z80_D5
- Z80-LOCAL_DATA1 pad 8: /RIO/Z80_D6 -> /Z80_D6
- Z80-LOCAL_DATA1 pad 9: /RIO/Z80_D7 -> /Z80_D7
- Z80-RIO_DATA1 pad 19: /RIO/ROM_D_RDY -> /RIO_CONTROL.ROM_RDY
- Z80-RIO_DATA1 pad 2: /RIO/Z80_D0 -> /Z80_D0
- Z80-RIO_DATA1 pad 3: /RIO/Z80_D1 -> /Z80_D1
- Z80-RIO_DATA1 pad 4: /RIO/Z80_D2 -> /Z80_D2
- Z80-RIO_DATA1 pad 5: /RIO/Z80_D3 -> /Z80_D3
- Z80-RIO_DATA1 pad 6: /RIO/Z80_D4 -> /Z80_D4
- Z80-RIO_DATA1 pad 7: /RIO/Z80_D5 -> /Z80_D5
- Z80-RIO_DATA1 pad 8: /RIO/Z80_D6 -> /Z80_D6
- Z80-RIO_DATA1 pad 9: /RIO/Z80_D7 -> /Z80_D7
- Z80_ADDRHIGH1 pad 2: /RIO/Z80_A8 -> /Z80_A8
- Z80_ADDRHIGH1 pad 3: /RIO/Z80_A9 -> /Z80_A9
- Z80_ADDRHIGH1 pad 4: /RIO/Z80_A10 -> /Z80_A10
- Z80_ADDRHIGH1 pad 5: /RIO/Z80_A11 -> /Z80_A11
- Z80_ADDRHIGH1 pad 6: /RIO/Z80_A12 -> /Z80_A12
- Z80_ADDRHIGH1 pad 7: /RIO/Z80_A13 -> /Z80_A13
- Z80_ADDRHIGH1 pad 8: /RIO/Z80_A14 -> /Z80_A14
- Z80_ADDRHIGH1 pad 9: /RIO/Z80_A15 -> /Z80_A15
- Z80_ADDRLOW1 pad 2: /RIO/Z80_A0 -> /Z80_A0
- Z80_ADDRLOW1 pad 3: /RIO/Z80_A1 -> /Z80_A1
- Z80_ADDRLOW1 pad 4: /RIO/Z80_A2 -> /Z80_A2
- Z80_ADDRLOW1 pad 5: /RIO/Z80_A3 -> /Z80_A3
- Z80_ADDRLOW1 pad 6: /RIO/Z80_A4 -> /Z80_A4
- Z80_ADDRLOW1 pad 7: /RIO/Z80_A5 -> /Z80_A5
- Z80_ADDRLOW1 pad 8: /RIO/Z80_A6 -> /Z80_A6
- Z80_ADDRLOW1 pad 9: /RIO/Z80_A7 -> /Z80_A7

Commit message: KiCAD PCB layout testing
Parts:
- removed CACHE1: AS6C1008-55PCN, Package_DIP:DIP-32_W15.24mm_Socket
- removed D13, D14, D15: 1N4148, Diode_THT:D_T-1_P5.08mm_Horizontal
- removed IC11, IC12: 74590N, Package_DIP:DIP-16_W7.62mm_Socket
- removed J10: Logic core connector (main), Connector_PinHeader_2.54mm:PinHeader_2x40_P2.54mm_Vertical
- removed R10, R11: 10K, Resistor_THT:R_Axial_DIN0207_L6.3mm_D2.5mm_P10.16mm_Horizontal
- removed U1: FREENOVE_ESP32-WROVER-DEV, esp32-wrover:FREENOVE_ESP32-WROVER-DEV
- added CACHE3: AS6C1008-55PCN, Package_DIP:DIP-32_W15.24mm, F.Cu at (144.1, 69.2)
- added D17: 1N4148, Diode_THT:D_T-1_P5.08mm_Horizontal, F.Cu at (115.0, 77.0)
- added D18: 1N4148, Diode_THT:D_T-1_P5.08mm_Horizontal, F.Cu at (133.0, 144.0)
- added D3: 1N4148, Diode_THT:D_T-1_P5.08mm_Horizontal, F.Cu at (121.0, 144.0)
- added D4: 1N4148, Diode_THT:D_T-1_P5.08mm_Horizontal, F.Cu at (213.0, 38.0)
- added D6: 1N4148, Diode_THT:D_T-1_P5.08mm_Horizontal, F.Cu at (80.0, 150.0)
- added DIAG-ESP_CONTROL1: PinHeader_2.54mm, Connector_PinHeader_2.54mm:PinHeader_1x08_P2.54mm_Vertical, F.Cu at (54.0, 44.5)
- added DIAG-ESP_SPI1: PinHeader_2.54mm, Connector_PinHeader_2.54mm:PinHeader_1x08_P2.54mm_Vertical, F.Cu at (227.3, 36.2)
- added DIAG-LOCAL_ADD_HIGH1: PinHeader_2.54mm, Connector_PinHeader_2.54mm:PinHeader_1x08_P2.54mm_Vertical, F.Cu at (162.6, 125.7)
- added DIAG-LOCAL_ADD_LOW1: PinHeader_2.54mm, Connector_PinHeader_2.54mm:PinHeader_1x08_P2.54mm_Vertical, F.Cu at (108.0, 109.9)
- added DIAG-LOCAL_DATA1: PinHeader_2.54mm, Connector_PinHeader_2.54mm:PinHeader_1x08_P2.54mm_Vertical, F.Cu at (229.2, 130.8)
- added DIAG-Z80_CONTROL1: PinHeader_2.54mm, Connector_PinHeader_2.54mm:PinHeader_1x08_P2.54mm_Vertical, F.Cu at (109.2, 157.5)
- added ESP1: FREENOVE_ESP32-WROVER-DEV, esp32-wrover:FREENOVE_ESP32-WROVER-DEV, F.Cu at (248.9, 52.7)
- added EX_SPI1: PinSocket_2.54mm, Connector_PinSocket_2.54mm:PinSocket_1x06_P2.54mm_Vertical, F.Cu at (227.3, 63.5)
- added IC2: 74HC590N, Package_DIP:DIP-16_W7.62mm_Socket, F.Cu at (90.8, 67.3)
- added IC3: 74HC590N, Package_DIP:DIP-16_W7.62mm_Socket, F.Cu at (191.8, 71.1)
- added J9: Logic core connector, Connector_PinHeader_2.54mm:PinHeader_2x25_P2.54mm_Vertical, F.Cu at (49.5, 154.3)
- added R15: R10K, Resistor_THT:R_Axial_DIN0207_L6.3mm_D2.5mm_P10.16mm_Horizontal, F.Cu at (129.0, 150.0)
- added R2: 22K, Resistor_THT:R_Axial_DIN0207_L6.3mm_D2.5mm_P10.16mm_Horizontal, F.Cu at (104.0, 144.0)
- ESP_CONTROL_DIRECTOR1: value 74244N -> 74HC244N
- IC1: value 7432N -> 74HC32N
- JP1: value PINHD-ADDR_FILTER -> PINHD-POWER/RESET
- JP2: value PINHD-POWER/RESET -> PINHD-ADDR_FILTER
- R5: value 22K -> 10K
- R8: value 1K -> 10K
- RIO1: footprint Package_DIP:DIP-32_W15.24mm_Socket -> Package_DIP:DIP-32_W15.24mm
- RIO_DECODER1, Z80-LOCAL_DATA1, Z80-RIO_DATA1, Z80_ADDRHIGH1, Z80_ADDRLOW1: value 74245N -> 74HC245N
- SPI-LOCAL_ADDR_L.IN1, SPI-LOCAL_ADD_H.IN1, SPI-LOCAL_DATA.IN1, SPI-Z80_CONTROL.IN1: value 74165N -> 74HC165N
- moved D7 180.2 mm to (71.0, 150.0)
- moved R3 159.1 mm to (93.0, 150.0)
- moved R4 158.5 mm to (59.1, 26.0)
- moved D8 156.1 mm to (99.0, 156.0)
- moved D9 139.3 mm to (74.0, 61.0)
- moved R5 138.6 mm to (200.0, 28.0), turned to 0 degrees
- moved D11 132.0 mm to (108.0, 150.0)
- moved R6 129.0 mm to (262.3, 87.6), turned to -90 degrees
- moved SPI-LOCAL_DATA.OUT1 104.7 mm to (76.8, 92.1)
- moved D12 103.8 mm to (46.0, 33.0), turned to 0 degrees
- moved LOCAL_DATA_BIAS1 103.7 mm to (71.8, 96.5)
- moved D5 98.4 mm to (121.0, 150.0), turned to 0 degrees
- moved SPI-LOCAL_DATA.IN1 88.6 mm to (244.5, 144.1), turned to 90 degrees
- moved JP1 85.4 mm to (59.0, 149.0), turned to 0 degrees
- moved RIO_DECODER1 85.0 mm to (196.9, 57.1), turned to 90 degrees
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Connections:
- net /Z80 BUS/VCC renamed /Z80 BUS/HOST VCC
- C1 pad 1: +5V -> Net-(D1-K)
- C2 pad 1: +5V -> Net-(D1-K)
- C3 pad 1: +5V -> Net-(D1-K)
- D1 pad 2: GND -> Net-(D1-A)
- D12 pad 1: /ESP_CONTROL.BUSRQ -> Net-(D12-K)
- D12 pad 2: /Z80_CONTROL.BUSRQ -> +5V
- D5 pad 1: Net-(D5-K) -> /Z80_CONTROL.BUSACK
- D5 pad 2: +5V -> /CORE/ESP_INT
- D7 pad 1: /Z80_CONTROL.WAIT -> /ESP_CONTROL.WAIT
- D7 pad 2: /CORE/ESP_INT -> /Z80_CONTROL.WAIT
- D8 pad 1: /CORE/Z80_HARDLOCK_RESET -> /ESP_CONTROL.ROMCS
- D8 pad 2: /CORE/ESP_INT -> /Z80_CONTROL.ROMCS
- D9 pad 1: /Z80_CONTROL.BUSACK -> /ESP_CONTROL.NMI
- D9 pad 2: /CORE/ESP_INT -> /Z80_CONTROL.NMI
- ESP_CONTROL_BIAS1 pad 1: Net-(D11-K) -> Net-(D12-K)
- ESP_CONTROL_DIRECTOR1 pad 1: /ESP_HARDLOCK -> /ESP_CONTROL.BUSRQ
- ESP_CONTROL_DIRECTOR1 pad 10: (no net) -> GND
- ESP_CONTROL_DIRECTOR1 pad 11: /ESP_CONTROL.RD -> /ESP_CONTROL.MEMRQ
- ESP_CONTROL_DIRECTOR1 pad 13: Net-(ESP_CONTROL_DIRECTOR1A-A2) -> /ESP_CONTROL.IORQ
- ESP_CONTROL_DIRECTOR1 pad 15: /ESP_CONTROL.IORQ -> /CORE/ESP_CONTROL.WR+ESP_PULSE
- ESP_CONTROL_DIRECTOR1 pad 17: /ESP_CONTROL.MEMRQ -> /ESP_CONTROL.RD
- ESP_CONTROL_DIRECTOR1 pad 19: /ESP_CONTROL.BUSRQ -> /ESP_HARDLOCK
- ESP_CONTROL_DIRECTOR1 pad 20: (no net) -> +5V
- ESP_CONTROL_DIRECTOR1 pad 3: /Z80_CONTROL.MEMRQ -> /Z80_CONTROL.RD
- ESP_CONTROL_DIRECTOR1 pad 4: Net-(ESP_CONTROL_DIRECTOR1A-A2) -> /CORE/ESP_CONTROL.WR+ESP_PULSE
- ESP_CONTROL_DIRECTOR1 pad 5: /Z80_CONTROL.IORQ -> /Z80_CONTROL.WR
- ESP_CONTROL_DIRECTOR1 pad 7: /Z80_CONTROL.WR -> /Z80_CONTROL.IORQ
- ESP_CONTROL_DIRECTOR1 pad 9: /Z80_CONTROL.RD -> /Z80_CONTROL.MEMRQ
- ESP_CONTROL_DIRECTOR_BIAS1 pad 1: Net-(D5-K) -> Net-(D10-K)
- IC1 pad 1: Net-(IC1A-I0) -> GND
- IC1 pad 10: /ESP_CONTROL.BUSRQ -> GND
- IC1 pad 11: Net-(ESP_CONTROL_DIRECTOR1A-A2) -> /CORE/ESP_CONTROL.WR+ESP_PULSE
- IC1 pad 14: (no net) -> +5V
- IC1 pad 2: /ESP_HARDLOCK -> GND
- IC1 pad 3: /Logic core/PRE_Z80_HARDLOCK -> unconnected-(IC1-Pad3)
- IC1 pad 4: /PERM_Z80_IORQ -> GND
- IC1 pad 5: /CACHE_DATASTATUS -> GND
- IC1 pad 6: /CACHE_CONTROL.DATASTATUS+PERM_Z80_IORQ -> unconnected-(IC1-Pad6)
- IC1 pad 7: (no net) -> GND
- IC1 pad 8: /Logic core/ESP_IOD_CONFIG -> unconnected-(IC1-Pad8)
- IC1 pad 9: Net-(IC1C-I0) -> GND
- JP1 pad 1: GND -> /Z80_CONTROL.RESET
- JP1 pad 2: /IORQ_FILTER_BIT -> GND
- JP1 pad 3: /Z80_A0 -> Net-(D1-K)
- JP2 pad 1: /Z80_CONTROL.RESET -> GND
- JP2 pad 2: GND -> /IORQ_FILTER_BIT
- JP2 pad 3: +5V -> /Z80_A0
- LOCAL_DATA_BIAS1 pad 1: Net-(D10-K) -> Net-(D11-K)
- R1 pad 1: Net-(D1-K) -> Net-(D1-A)
- R3 pad 1: +5V -> GND
- R4 pad 1: /CORE/ESP_INT -> +5V
- R4 pad 2: GND -> /CORE/ESP_SPI_INT.MR
- R5 pad 1: +5V -> Net-(RIO_DECODER1-A->B)
- R5 pad 2: /CORE/ESP_SPI_INT.MR -> +5V
- R6 pad 1: /CACHE_DATASTATUS -> +5V
- R6 pad 2: +5V -> /RIO/RIO_CE2
- R7 pad 1: Net-(RIO_DECODER1A-DIR) -> /CACHE_DATASTATUS
- R8 pad 1: /!CACHE_DATASTATUS -> /CACHE/CACHE_CE2
- RIO1 pad 29: /RIO/RIO_CONTROL.WE -> /RIO_CONTROL.WE
- RIO_DECODER1 pad 1: Net-(RIO_DECODER1A-DIR) -> Net-(RIO_DECODER1-A->B)
- RIO_DECODER1 pad 10: (no net) -> GND
- RIO_DECODER1 pad 20: (no net) -> +5V
- SPI-ESP_CONTROL.OUT1 pad 16: (no net) -> +5V
- SPI-ESP_CONTROL.OUT1 pad 8: (no net) -> GND
- SPI-LOCAL_ADDR_L.IN1 pad 10: Net-(SPI-LOCAL_ADDR_L.IN1A-SER) -> Net-(SPI-LOCAL_ADDR_L.IN1-DS)
- SPI-LOCAL_ADDR_L.IN1 pad 16: (no net) -> +5V
- SPI-LOCAL_ADDR_L.IN1 pad 7: unconnected-(SPI-LOCAL_ADDR_L.IN1A-~{QH}-Pad7) -> Net-(SPI-LOCAL_ADDR_L.IN1-~{Q7})
- SPI-LOCAL_ADDR_L.IN1 pad 8: (no net) -> GND
- SPI-LOCAL_ADDR_L.IN1 pad 9: Net-(SPI-LOCAL_ADDR_L.IN1A-QH) -> unconnected-(SPI-LOCAL_ADDR_L.IN1-Q7-Pad9)
- SPI-LOCAL_ADD_H.IN1 pad 10: Net-(SPI-LOCAL_ADDR_L.IN1A-QH) -> Net-(SPI-LOCAL_ADDR_L.IN1-~{Q7})
- SPI-LOCAL_ADD_H.IN1 pad 16: (no net) -> +5V
- SPI-LOCAL_ADD_H.IN1 pad 7: unconnected-(SPI-LOCAL_ADD_H.IN1A-~{QH}-Pad7) -> /CORE/ESP_SPI_INT.MISO
- SPI-LOCAL_ADD_H.IN1 pad 8: (no net) -> GND
- SPI-LOCAL_ADD_H.IN1 pad 9: /CORE/ESP_SPI_INT.MISO -> unconnected-(SPI-LOCAL_ADD_H.IN1-Q7-Pad9)
- SPI-LOCAL_ADD_HIGH.OUT1 pad 16: (no net) -> +5V
- SPI-LOCAL_ADD_HIGH.OUT1 pad 8: (no net) -> GND
- SPI-LOCAL_ADD_L.OUT1 pad 16: (no net) -> +5V
- SPI-LOCAL_ADD_L.OUT1 pad 8: (no net) -> GND
- SPI-LOCAL_DATA.IN1 pad 16: (no net) -> +5V
- SPI-LOCAL_DATA.IN1 pad 7: unconnected-(SPI-LOCAL_DATA.IN1A-~{QH}-Pad7) -> Net-(SPI-LOCAL_DATA.IN1-~{Q7})
- SPI-LOCAL_DATA.IN1 pad 8: (no net) -> GND
- SPI-LOCAL_DATA.IN1 pad 9: Net-(SPI-LOCAL_DATA.IN1A-QH) -> unconnected-(SPI-LOCAL_DATA.IN1-Q7-Pad9)
- SPI-LOCAL_DATA.OUT1 pad 16: (no net) -> +5V
- SPI-LOCAL_DATA.OUT1 pad 8: (no net) -> GND
- SPI-Z80_CONTROL.IN1 pad 10: Net-(SPI-LOCAL_DATA.IN1A-QH) -> Net-(SPI-LOCAL_DATA.IN1-~{Q7})
- SPI-Z80_CONTROL.IN1 pad 16: (no net) -> +5V
- SPI-Z80_CONTROL.IN1 pad 7: unconnected-(SPI-Z80_CONTROL.IN1A-~{QH}-Pad7) -> Net-(SPI-LOCAL_ADDR_L.IN1-DS)
- SPI-Z80_CONTROL.IN1 pad 8: (no net) -> GND
- SPI-Z80_CONTROL.IN1 pad 9: Net-(SPI-LOCAL_ADDR_L.IN1A-SER) -> unconnected-(SPI-Z80_CONTROL.IN1-Q7-Pad9)
- Z80-LOCAL_DATA1 pad 10: (no net) -> GND
- Z80-LOCAL_DATA1 pad 20: (no net) -> +5V
- Z80-RIO_DATA1 pad 10: (no net) -> GND
- Z80-RIO_DATA1 pad 20: (no net) -> +5V
- Z80_ADDRHIGH1 pad 10: (no net) -> GND
- Z80_ADDRHIGH1 pad 20: (no net) -> +5V
- Z80_ADDRLOW1 pad 10: (no net) -> GND
- Z80_ADDRLOW1 pad 20: (no net) -> +5V
Other:
- board size 239.3 x 158.4 mm -> 236.8 x 145 mm

Commit message: KiCad close but failed attempt at PCB
Parts:
- removed D17, D18: 1N4148, Diode_THT:D_T-1_P5.08mm_Horizontal
- removed DIAG-ESP_SPI1: PinHeader_2.54mm, Connector_PinHeader_2.54mm:PinHeader_1x08_P2.54mm_Vertical
- removed R15: R10K, Resistor_THT:R_Axial_DIN0207_L6.3mm_D2.5mm_P10.16mm_Horizontal
- moved D4 153.8 mm to (86.5, 125.5), turned to 180 degrees
- moved ESP_CONTROL_DIRECTOR_BIAS1 150.7 mm to (143.0, 48.2)
- moved SPI-LOCAL_DATA.IN1 126.8 mm to (120.4, 118.1)
- moved J9 117.9 mm to (123.2, 62.2), turned to 90 degrees
- moved D10 117.8 mm to (138.5, 48.2), turned to 180 degrees
- moved SPI-LOCAL_DATA.OUT1 94.1 mm to (164.5, 126.3), turned to 0 degrees
- moved LOCAL_DATA_BIAS1 91.7 mm to (160.1, 121.2), turned to -90 degrees
- moved D7 88.0 mm to (100.5, 67.1), turned to -90 degrees
- moved D2 80.2 mm to (95.5, 117.8)
- moved IC1 78.2 mm to (92.7, 127.1)
- moved R4 74.6 mm to (130.3, 48.2), turned to 180 degrees
- moved R7 65.6 mm to (140.0, 91.5), turned to 90 degrees
- moved R5 65.1 mm to (212.1, 92.0)
- moved D11 63.4 mm to (164.5, 121.2)
- moved JP1 58.9 mm to (117.9, 147.9)
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Other:
- board size 236.8 x 145 mm -> 180 x 120 mm
