File: KiCad7/FujiNet_Z80Bus_Modules/GLUE_ZXspectrum/GLUE_ZXspectrum_connectors.kicad_sch (KiCad schematic)
At the start: 2 parts, among them J12 Conn_02x12_Odd_Even, J3 Conn_02x12_Odd_Even

Commit message: GLUE is broken again, logic gate annotation issue
Parts:
- renumbered J3 to J1, J12 to J2
Changed lines of the file:
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@@
   (symbol (lib_id "Connector_Generic:Conn_02x12_Odd_Even") (at 137.795 53.34 0) (unit 1)
     (in_bom yes) (on_board yes) (dnp no)
-    (property "Reference" "J3" (at 139.065 38.1 0)
+    (property "Reference" "J1" (at 139.065 38.1 0)
       (effects (font (size 1.27 1.27)))
     )
@@
     (pin "9")
     (instances
-      (project "FujiNet_Z80Bus_ReferenceDesign"
-        (path "/532c0392-800e-45cc-8170-6d32f2390e83/15e820a2-e197-4611-93bc-baa539eede01"
-          (reference "J3") (unit 1)
+      (project "GLUE_ZXspectrum_impl"
+        (path "/532c0392-800e-45cc-8170-6d32f2390e83/0da5b4c6-619f-4cd1-829e-b9ad71c924a4/38b7d772-cf38-4194-8e0b-ce11c179768d"
+          (reference "J1") (unit 1)
         )
-        (path "/532c0392-800e-45cc-8170-6d32f2390e83/6a1fd481-1635-4a64-b244-c204161ad407/38b7d772-cf38-4194-8e0b-ce11c179768d"
-          (reference "J?") (unit 1)
+      )
+      (project "GLUE_ZXspectrum"
+        (path "/648e0b91-567a-4972-a379-57b42123c6d5/38b7d772-cf38-4194-8e0b-ce11c179768d"
+          (reference "J1") (unit 1)
         )
       )
@@
   (symbol (lib_id "Connector_Generic:Conn_02x12_Odd_Even") (at 138.43 99.695 0) (unit 1)
     (in_bom yes) (on_board yes) (dnp no) (fields_autoplaced)
-    (property "Reference" "J12" (at 139.7 81.28 0)
+    (property "Reference" "J2" (at 139.7 81.28 0)
       (effects (font (size 1.27 1.27)))
     )
@@
     (pin "9")
     (instances
-      (project "FujiNet_Z80Bus_ReferenceDesign"
-        (path "/532c0392-800e-45cc-8170-6d32f2390e83/15e820a2-e197-4611-93bc-baa539eede01"
-          (reference "J12") (unit 1)
+      (project "GLUE_ZXspectrum_impl"
+        (path "/532c0392-800e-45cc-8170-6d32f2390e83/0da5b4c6-619f-4cd1-829e-b9ad71c924a4/38b7d772-cf38-4194-8e0b-ce11c179768d"
+          (reference "J2") (unit 1)
         )
-        (path "/532c0392-800e-45cc-8170-6d32f2390e83/6a1fd481-1635-4a64-b244-c204161ad407/38b7d772-cf38-4194-8e0b-ce11c179768d"
-          (reference "J?") (unit 1)
+      )
+      (project "GLUE_ZXspectrum"
+        (path "/648e0b91-567a-4972-a379-57b42123c6d5/38b7d772-cf38-4194-8e0b-ce11c179768d"
+          (reference "J2") (unit 1)
         )
       )
@@
   (symbol (lib_id "power:GND") (at 88.9 114.935 0) (mirror y) (unit 1)
     (in_bom yes) (on_board yes) (dnp no) (fields_autoplaced)
-    (property "Reference" "#PWR072" (at 88.9 121.285 0)
+    (property "Reference" "#PWR08" (at 88.9 121.285 0)
       (effects (font (size 1.27 1.27)) hide)
     )
@@
     (pin "1")
     (instances
-      (project "FujiNet_Z80Bus_ReferenceDesign"
-        (path "/532c0392-800e-45cc-8170-6d32f2390e83/15e820a2-e197-4611-93bc-baa539eede01"
-          (reference "#PWR072") (unit 1)
-        )
-        (path "/532c0392-800e-45cc-8170-6d32f2390e83/6a1fd481-1635-4a64-b244-c204161ad407/38b7d772-cf38-4194-8e0b-ce11c179768d"
-          (reference "#PWR?") (unit 1)
+      (project "GLUE_ZXspectrum_impl"
+        (path "/532c0392-800e-45cc-8170-6d32f2390e83/0da5b4c6-619f-4cd1-829e-b9ad71c924a4/38b7d772-cf38-4194-8e0b-ce11c179768d"
+          (reference "#PWR08") (unit 1)
         )
       )
       (project "GLUE_ZXspectrum"
         (path "/648e0b91-567a-4972-a379-57b42123c6d5/38b7d772-cf38-4194-8e0b-ce11c179768d"
-          (reference "#PWR078") (unit 1)
+          (reference "#PWR015") (unit 1)
         )
       )
@@
   (symbol (lib_id "power:+5V") (at 88.9 112.395 0) (mirror y) (unit 1)
     (in_bom yes) (on_board yes) (dnp no) (fields_autoplaced)
-    (property "Reference" "#PWR071" (at 88.9 116.205 0)
+    (property "Reference" "#PWR07" (at 88.9 116.205 0)
       (effects (font (size 1.27 1.27)) hide)
     )
@@
     (pin "1")
     (instances
-      (project "FujiNet_Z80Bus_ReferenceDesign"
-        (path "/532c0392-800e-45cc-8170-6d32f2390e83/15e820a2-e197-4611-93bc-baa539eede01"
-          (reference "#PWR071") (unit 1)
-        )
-        (path "/532c0392-800e-45cc-8170-6d32f2390e83/6a1fd481-1635-4a64-b244-c204161ad407/38b7d772-cf38-4194-8e0b-ce11c179768d"
-          (reference "#PWR?") (unit 1)
+      (project "GLUE_ZXspectrum_impl"
+        (path "/532c0392-800e-45cc-8170-6d32f2390e83/0da5b4c6-619f-4cd1-829e-b9ad71c924a4/38b7d772-cf38-4194-8e0b-ce11c179768d"
+          (reference "#PWR07") (unit 1)
         )
       )
       (project "GLUE_ZXspectrum"
         (path "/648e0b91-567a-4972-a379-57b42123c6d5/38b7d772-cf38-4194-8e0b-ce11c179768d"
-          (reference "#PWR077") (unit 1)
+          (reference "#PWR014") (unit 1)
         )
       )

Commit message: KiCad FIXED GLUE
Parts:
- removed J1, J2: Conn_02x12_Odd_Even, Connector_PinHeader_2.54mm:PinHeader_2x16_P2.54mm_Vertical, symbol Connector_Generic:Conn_02x12_Odd_Even
- added J1: Conn_01x24_Socket, Connector_PinSocket_2.54mm:PinSocket_1x24_P2.54mm_Vertical, symbol Connector:Conn_01x24_Socket
- added J2: Conn_01x26_Socket, Connector_PinSocket_2.54mm:PinSocket_1x26_P2.54mm_Vertical, symbol Connector:Conn_01x26_Socket
Connections:
- net !ESP_HARDLOCK: now also J2.21 (Pin_21)
- net !Z80_HARDLOCK: now also J2.23 (Pin_23)
- net +5V: now also J2.1 (Pin_1)
- net CACHE_CONTROL.A16: now also J1.14 (Pin_14)
- net CACHE_CONTROL.CS: now also J1.17 (Pin_17)
- net CACHE_CONTROL.DATASTATUS+PERM_Z80_IORQ: now also J1.13 (Pin_13)
- net CACHE_CONTROL.OE: now also J1.16 (Pin_16)
- net CACHE_CONTROL.WE: now also J1.15 (Pin_15)
- net CACHE_DATASTATUS: now also J1.5 (Pin_5)
- net ESP_CONTROL.BUSRQ: now also J2.15 (Pin_15)
- net ESP_CONTROL.IORQ: now also J2.13 (Pin_13)
- net ESP_CONTROL.MEMRQ: now also J2.14 (Pin_14)
- net ESP_CONTROL.ROMCS: now also J2.16 (Pin_16)
- net ESP_CONTROL.WR: now also J2.12 (Pin_12)
- net ESP_HARDLOCK: now also J2.20 (Pin_20)
- net ESP_ROMSEL_0: now also J2.18 (Pin_18)
- net ESP_ROMSEL_1: now also J2.19 (Pin_19)
- net ESP_ROM_WR_PROTECT: now also J2.17 (Pin_17)
- net ESP_WAIT_RESET: now also J1.6 (Pin_6)
- net GND: now also J2.26 (Pin_26)
- net IORQ_FILTER_BIT: now also J1.1 (Pin_1)
- net LOCAL_CONTROL.IORQ: now also J2.10 (Pin_10)
- net LOCAL_CONTROL.MEMRQ: now also J2.11 (Pin_11)
- net LOCAL_CONTROL.RD: now also J2.8 (Pin_8)
- net LOCAL_CONTROL.WR: now also J2.9 (Pin_9)
- net PERM_Z80_IORQ: now also J2.24 (Pin_24)
- net RIO_CONTROL.A14: now also J1.20 (Pin_20)
- net RIO_CONTROL.A15: now also J1.19 (Pin_19)
- net RIO_CONTROL.OE: now also J1.22 (Pin_22)
- net RIO_CONTROL.WE: now also J1.21 (Pin_21)
- net WAIT_IO: now also J1.4 (Pin_4)
- net Z80_A14: now also J1.7 (Pin_7)
- net Z80_A15: now also J1.8 (Pin_8)
- net Z80_BUS_CONTROL.Z80_ADD_DIR: now also J1.10 (Pin_10)
- net Z80_BUS_CONTROL.Z80_ADD_OE: now also J1.9 (Pin_9)
- net Z80_BUS_CONTROL.Z80_DATA_DIR: now also J1.11 (Pin_11)
- net Z80_BUS_CONTROL.Z80_DATA_OE: now also J1.12 (Pin_12)
- net Z80_CONTROL.BUSRQ: now also J2.6 (Pin_6)
- net Z80_CONTROL.IORQ: now also J2.4 (Pin_4)
- net Z80_CONTROL.MEMRQ: now also J2.5 (Pin_5)
- net Z80_CONTROL.RD: now also J2.2 (Pin_2)
- net Z80_CONTROL.WAIT: now also J2.7 (Pin_7)
- net Z80_CONTROL.WR: now also J2.3 (Pin_3)
- net Z80_HARDLOCK: now also J2.22 (Pin_22)
- net Z80_HARDLOCK_RESET: now also J1.3 (Pin_3)
- net Z80_HARDLOCK_SET: now also J1.2 (Pin_2)
- new net RIO_CONTROL.A16: J1.18 (Pin_18)
- new net RIO_CONTROL.CE: J1.23 (Pin_23)
- new net RIO_CONTROL.ROM_RDY: J1.24 (Pin_24)
- no-connect marks 2 -> 1
