File: KiCad7/FujiNet_Z80Bus_Modules/GLUE_ZXspectrum/CACHE CONTROL.kicad_sch (KiCad schematic)
At the start: 2 parts, among them IC1 74HC32N, IC10 74HC08N

Commit message: KiCad FIXED GLUE
Parts:
- renumbered IC10 to IC?, IC1 to IC?
Changed lines of the file:
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@@
   (symbol (lib_id "74xx:74LS08") (at 147.32 115.57 0) (unit 4)
     (in_bom yes) (on_board yes) (dnp no)
-    (property "Reference" "IC10" (at 149.86 111.76 0)
+    (property "Reference" "IC?" (at 149.86 111.76 0)
       (effects (font (size 1.4986 1.4986)) (justify left bottom))
     )
@@
       (project "FujiNet_Z80Bus_Basic"
         (path "/35e54075-8ed7-4bf6-837e-479a97e77d5d/344f9fe5-9c02-46d6-8016-81558291d94c"
-          (reference "IC10") (unit 4)
-        )
-      )
-      (project "GLUE_ZXspectrum_impl"
-        (path "/532c0392-800e-45cc-8170-6d32f2390e83"
           (reference "IC?") (unit 4)
         )
-        (path "/532c0392-800e-45cc-8170-6d32f2390e83/0da5b4c6-619f-4cd1-829e-b9ad71c924a4/93c14a9e-4a71-4950-b006-2a9affe18130"
-          (reference "IC4") (unit 4)
-        )
-      )
-      (project "GLUE_ZXspectrum"
-        (path "/648e0b91-567a-4972-a379-57b42123c6d5/93c14a9e-4a71-4950-b006-2a9affe18130"
+      )
+      (project "GLUE_ZXspectrum_impl"
+        (path "/532c0392-800e-45cc-8170-6d32f2390e83"
+          (reference "IC?") (unit 4)
+        )
+        (path "/532c0392-800e-45cc-8170-6d32f2390e83/0da5b4c6-619f-4cd1-829e-b9ad71c924a4/93c14a9e-4a71-4950-b006-2a9affe18130"
           (reference "IC8") (unit 4)
         )
       )
+      (project "GLUE_ZXspectrum"
+        (path "/648e0b91-567a-4972-a379-57b42123c6d5/93c14a9e-4a71-4950-b006-2a9affe18130"
+          (reference "IC?") (unit 4)
+        )
+      )
     )
   )
   (symbol (lib_id "74xx:74LS08") (at 147.32 104.14 0) (unit 3)
     (in_bom yes) (on_board yes) (dnp no)
-    (property "Reference" "IC10" (at 149.86 100.33 0)
+    (property "Reference" "IC?" (at 149.86 100.33 0)
       (effects (font (size 1.4986 1.4986)) (justify left bottom))
     )
@@
       (project "FujiNet_Z80Bus_Basic"
         (path "/35e54075-8ed7-4bf6-837e-479a97e77d5d/344f9fe5-9c02-46d6-8016-81558291d94c"
-          (reference "IC10") (unit 3)
-        )
-      )
-      (project "GLUE_ZXspectrum_impl"
-        (path "/532c0392-800e-45cc-8170-6d32f2390e83"
           (reference "IC?") (unit 3)
         )
-        (path "/532c0392-800e-45cc-8170-6d32f2390e83/0da5b4c6-619f-4cd1-829e-b9ad71c924a4/93c14a9e-4a71-4950-b006-2a9affe18130"
-          (reference "IC4") (unit 3)
-        )
-      )
-      (project "GLUE_ZXspectrum"
-        (path "/648e0b91-567a-4972-a379-57b42123c6d5/93c14a9e-4a71-4950-b006-2a9affe18130"
+      )
+      (project "GLUE_ZXspectrum_impl"
+        (path "/532c0392-800e-45cc-8170-6d32f2390e83"
+          (reference "IC?") (unit 3)
+        )
+        (path "/532c0392-800e-45cc-8170-6d32f2390e83/0da5b4c6-619f-4cd1-829e-b9ad71c924a4/93c14a9e-4a71-4950-b006-2a9affe18130"
           (reference "IC8") (unit 3)
         )
       )
+      (project "GLUE_ZXspectrum"
+        (path "/648e0b91-567a-4972-a379-57b42123c6d5/93c14a9e-4a71-4950-b006-2a9affe18130"
+          (reference "IC?") (unit 3)
+        )
+      )
     )
   )
   (symbol (lib_id "74xx:74LS32") (at 147.32 69.85 0) (mirror x) (unit 2)
     (in_bom yes) (on_board yes) (dnp no)
-    (property "Reference" "IC1" (at 149.86 64.77 0)
+    (property "Reference" "IC?" (at 149.86 64.77 0)
       (effects (font (size 1.4986 1.4986)) (justify left bottom))
     )
@@
       (project "FujiNet_Z80Bus_Basic"
         (path "/35e54075-8ed7-4bf6-837e-479a97e77d5d/344f9fe5-9c02-46d6-8016-81558291d94c"
-          (reference "IC1") (unit 2)
-        )
-      )
-      (project "GLUE_ZXspectrum_impl"
-        (path "/532c0392-800e-45cc-8170-6d32f2390e83"
-          (reference "IC?") (unit 2)
-        )
-        (path "/532c0392-800e-45cc-8170-6d32f2390e83/0da5b4c6-619f-4cd1-829e-b9ad71c924a4/93c14a9e-4a71-4950-b006-2a9affe18130"
-          (reference "IC14") (unit 2)
-        )
-      )
-      (project "GLUE_ZXspectrum"
-        (path "/648e0b91-567a-4972-a379-57b42123c6d5/93c14a9e-4a71-4950-b006-2a9affe18130"
-          (reference "IC7") (unit 2)
+          (reference "IC?") (unit 2)
+        )
+      )
+      (project "GLUE_ZXspectrum_impl"
+        (path "/532c0392-800e-45cc-8170-6d32f2390e83"
+          (reference "IC?") (unit 2)
+        )
+        (path "/532c0392-800e-45cc-8170-6d32f2390e83/0da5b4c6-619f-4cd1-829e-b9ad71c924a4/93c14a9e-4a71-4950-b006-2a9affe18130"
+          (reference "IC5") (unit 2)
+        )
+      )
+      (project "GLUE_ZXspectrum"
+        (path "/648e0b91-567a-4972-a379-57b42123c6d5/93c14a9e-4a71-4950-b006-2a9affe18130"
+          (reference "IC?") (unit 2)
         )
       )
@@
   (symbol (lib_id "74xx:74LS08") (at 147.32 81.28 0) (unit 1)
     (in_bom yes) (on_board yes) (dnp no)
-    (property "Reference" "IC10" (at 149.86 77.47 0)
+    (property "Reference" "IC?" (at 149.86 77.47 0)
       (effects (font (size 1.4986 1.4986)) (justify left bottom))
     )
@@
       (project "FujiNet_Z80Bus_Basic"
         (path "/35e54075-8ed7-4bf6-837e-479a97e77d5d/344f9fe5-9c02-46d6-8016-81558291d94c"
-          (reference "IC10") (unit 1)
-        )
-      )
-      (project "GLUE_ZXspectrum_impl"
-        (path "/532c0392-800e-45cc-8170-6d32f2390e83"
           (reference "IC?") (unit 1)
         )
-        (path "/532c0392-800e-45cc-8170-6d32f2390e83/0da5b4c6-619f-4cd1-829e-b9ad71c924a4/93c14a9e-4a71-4950-b006-2a9affe18130"
-          (reference "IC4") (unit 1)
-        )
-      )
-      (project "GLUE_ZXspectrum"
-        (path "/648e0b91-567a-4972-a379-57b42123c6d5/93c14a9e-4a71-4950-b006-2a9affe18130"
+      )
+      (project "GLUE_ZXspectrum_impl"
+        (path "/532c0392-800e-45cc-8170-6d32f2390e83"
+          (reference "IC?") (unit 1)
+        )
+        (path "/532c0392-800e-45cc-8170-6d32f2390e83/0da5b4c6-619f-4cd1-829e-b9ad71c924a4/93c14a9e-4a71-4950-b006-2a9affe18130"
           (reference "IC8") (unit 1)
         )
       )
+      (project "GLUE_ZXspectrum"
+        (path "/648e0b91-567a-4972-a379-57b42123c6d5/93c14a9e-4a71-4950-b006-2a9affe18130"
+          (reference "IC?") (unit 1)
+        )
+      )
     )
   )
   (symbol (lib_id "74xx:74LS08") (at 147.32 92.71 0) (unit 2)
     (in_bom yes) (on_board yes) (dnp no)
-    (property "Reference" "IC10" (at 149.86 88.9 0)
+    (property "Reference" "IC?" (at 149.86 88.9 0)
       (effects (font (size 1.4986 1.4986)) (justify left bottom))
     )
@@
       (project "FujiNet_Z80Bus_Basic"
         (path "/35e54075-8ed7-4bf6-837e-479a97e77d5d/344f9fe5-9c02-46d6-8016-81558291d94c"
-          (reference "IC10") (unit 2)
-        )
-      )
-      (project "GLUE_ZXspectrum_impl"
-        (path "/532c0392-800e-45cc-8170-6d32f2390e83"
-          (reference "IC?") (unit 2)
-        )
-        (path "/532c0392-800e-45cc-8170-6d32f2390e83/0da5b4c6-619f-4cd1-829e-b9ad71c924a4/93c14a9e-4a71-4950-b006-2a9affe18130"
-          (reference "IC4") (unit 2)
-        )
-      )
-      (project "GLUE_ZXspectrum"
-        (path "/648e0b91-567a-4972-a379-57b42123c6d5/93c14a9e-4a71-4950-b006-2a9affe18130"
+          (reference "IC?") (unit 2)
+        )
+      )
+      (project "GLUE_ZXspectrum_impl"
+        (path "/532c0392-800e-45cc-8170-6d32f2390e83"
+          (reference "IC?") (unit 2)
+        )
+        (path "/532c0392-800e-45cc-8170-6d32f2390e83/0da5b4c6-619f-4cd1-829e-b9ad71c924a4/93c14a9e-4a71-4950-b006-2a9affe18130"
           (reference "IC8") (unit 2)
         )
       )
+      (project "GLUE_ZXspectrum"
+        (path "/648e0b91-567a-4972-a379-57b42123c6d5/93c14a9e-4a71-4950-b006-2a9affe18130"
+          (reference "IC?") (unit 2)
+        )
+      )
