File: KiCad7/FujiNet_Z80Bus_Modules/GLUE_ZXspectrum/GLUE_ZXspectrum.kicad_sch (KiCad schematic)
At the start: 26 parts, among them IC1 74HC32N, IC10 74HC08N, IC2 7404N, IC3 7474N, IC4 74HC08N, IC7 74HC32N, IC8 74HC32N, IC9 74HC08N

Commit message: GLUE is broken again, logic gate annotation issue
Parts:
- removed IC1 (x5): 74HC32N, Package_DIP:DIP-14_W7.62mm_Socket, symbol 74xx:74LS32
- removed IC2: 7404N, Package_DIP:DIP-14_W7.62mm_Socket, symbol 74xx:74HC04
- removed IC4 (x2): 74HC08N, Package_DIP:DIP-14_W7.62mm_Socket, symbol 74xx:74LS08
- added IC10, IC? (x3): 74HC32N, Package_DIP:DIP-14_W7.62mm_Socket, symbol 74xx:74LS32
- added IC7: 7404N, Package_DIP:DIP-14_W7.62mm_Socket, symbol 74xx:74HC04
- added IC9: 74HC08N, Package_DIP:DIP-14_W7.62mm_Socket, symbol 74xx:74LS08
- renumbered C5 to C?, C4 to C?, D6 to D?, IC9 to IC1, IC8 to IC2, IC10 to IC?, IC2 to IC?, IC4 to IC?, IC7 to IC?, IC3 to IC?, IC1 to IC?, R2 to R?
Connections:
- net +5V: now also IC1.14 (VCC), IC2.14 (VCC), IC10.14 (VCC)
- net GND: now also IC1.7 (GND), IC2.7 (GND), IC10.10, IC10.7 (GND), IC10.9, IC7.11, IC9.10, IC9.12, IC9.13, IC9.9, IC?.1, IC?.10, IC?.10, IC?.2, IC?.9, IC?.9
Other:
- moved on the sheet: IC?A

Commit message: KiCad FIXED GLUE
Parts:
- removed IC1, IC9, IC? (x2): 74HC08N, Package_DIP:DIP-14_W7.62mm_Socket, symbol 74xx:74LS08
- removed IC10, IC2, IC? (x6): 74HC32N, Package_DIP:DIP-14_W7.62mm_Socket, symbol 74xx:74LS32
- removed IC7, IC?: 7404N, Package_DIP:DIP-14_W7.62mm_Socket, symbol 74xx:74HC04
- removed IC?: 7474N, Package_DIP:DIP-14_W7.62mm_Socket, symbol 74xx:74HC74
Connections:
- no-connect marks 12 -> 5
Other:
- removed sheet GLUE_ZXspectrum_connectors
