File: KiCad7/FujiNet_Z80Bus_Modules/IOCACHE-128K_ZXspectrum/IOCACHE-128k_ZXspectrum_impl/IOCACHE-128k_ZXspectrum_impl.kicad_pcb (KiCad board)
At the start: 2 copper layers, 0 parts

Commit message: KiCad IOCACHE_impl
Parts:
- added CACHE1: AS6C1008-55PCN, Package_DIP:DIP-32_W15.24mm_Socket, F.Cu at (129.8, 93.6)
- added IC1: 74HC590N, Package_DIP:DIP-16_W7.62mm_Socket, F.Cu at (133.0, 104.1)
- added IC2: 74HC590N, Package_DIP:DIP-16_W7.62mm_Socket, F.Cu at (156.0, 104.1)
- added J1: Conn_01x14_Socket, Connector_PinSocket_2.54mm:PinSocket_1x14_P2.54mm_Vertical, F.Cu at (179.0, 67.0)
- added J2: Conn_01x24_Socket, Connector_PinSocket_2.54mm:PinSocket_1x24_P2.54mm_Vertical, F.Cu at (119.0, 67.0)
- added R1: 10K, Resistor_THT:R_Axial_DIN0207_L6.3mm_D2.5mm_P10.16mm_Horizontal, F.Cu at (140.0, 69.1)
Routing:
- net +5V: track 0.00 -> 123.0 mm
- net /IOCACHE-128K_ZXspectrum/LOCAL_A11: track 0.00 -> 101.3 mm, vias 0 -> 1
- net /IOCACHE-128K_ZXspectrum/LOCAL_A8: track 0.00 -> 99.2 mm, vias 0 -> 1
- net /IOCACHE-128K_ZXspectrum/LOCAL_A9: track 0.00 -> 98.7 mm
- net /IOCACHE-128K_ZXspectrum/LOCAL_A10: track 0.00 -> 95.0 mm
- net GND: track 0.00 -> 79.1 mm, vias 0 -> 1
- net /IOCACHE-128K_ZXspectrum/CACHE_CONTROL.DATASTATUS+PERM_Z80_IORQ: track 0.00 -> 73.2 mm, vias 0 -> 1
- net /IOCACHE-128K_ZXspectrum/Z80_HARDLOCK: track 0.00 -> 69.9 mm
- net /IOCACHE-128K_ZXspectrum/CACHE_CONTROL.A16: track 0.00 -> 69.7 mm, vias 0 -> 1
- net /IOCACHE-128K_ZXspectrum/CACHE_DATASTATUS: track 0.00 -> 67.7 mm
- net /IOCACHE-128K_ZXspectrum/LOCAL_A0: track 0.00 -> 63.9 mm
- net /IOCACHE-128K_ZXspectrum/LOCAL_D1: track 0.00 -> 56.8 mm
- net /IOCACHE-128K_ZXspectrum/LOCAL_D2: track 0.00 -> 55.7 mm, vias 0 -> 1
- net /IOCACHE-128K_ZXspectrum/LOCAL_A7: track 0.00 -> 54.5 mm
- net /IOCACHE-128K_ZXspectrum/LOCAL_D0: track 0.00 -> 54.0 mm, vias 0 -> 1
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Other:
- board outline added: 70 x 67 mm
