File: KiCad7/FujiNet_Z80Bus_Modules/IOCACHE-128K_ZXspectrum/IOCACHE-128k_ZXspectrum_impl/IOCACHE-128k_ZXspectrum_impl.kicad_sch (KiCad schematic)
At the start: 0 parts

Commit message: KiCad IOCACHE_impl
Other:
- added sheet IOCACHE-128K_ZXspectrum (../IOCACHE-128K_ZXspectrum.kicad_sch)
Changed lines of the file:
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@@
   )
   (bus_alias "Z80_CONTROL" (members "Z80_CONTROL.RD" "Z80_CONTROL.WR" "Z80_CONTROL.IORQ" "Z80_CONTROL.MEMRQ" "Z80_CONTROL.BUSRQ" "Z80_CONTROL.WAIT" "Z80_CONTROL.ROMCS" "Z80_CONTROL.BUSACK" "Z80_CONTROL.NMI" "Z80_CONTROL.RESET"))
+  (sheet (at 102.235 34.29) (size 33.655 50.165) (fields_autoplaced)
+    (stroke (width 0.1524) (type solid))
+    (fill (color 0 0 0 0.0000))
+    (property "Sheetname" "IOCACHE-128K_ZXspectrum" (at 102.235 33.5784 0)
+      (effects (font (size 1.27 1.27)) (justify left bottom))
+    )
+    (property "Sheetfile" "../IOCACHE-128K_ZXspectrum.kicad_sch" (at 102.235 85.0396 0)
+      (effects (font (size 1.27 1.27)) (justify left top))
+    )
+    (pin "Z80_HARDLOCK" input (at 102.235 39.37 180)
+      (effects (font (size 1.27 1.27)) (justify left))
+    )
+    (pin "CACHE_DATASTATUS" input (at 102.235 43.18 180)
+      (effects (font (size 1.27 1.27)) (justify left))
+    )
+    (pin "{CACHE_CONTROL}" input (at 102.235 71.755 180)
+      (effects (font (size 1.27 1.27)) (justify left))
+    )
+    (pin "CACHE_SEL_1" input (at 102.235 46.99 180)
+      (effects (font (size 1.27 1.27)) (justify left))
+    )
+    (pin "CACHE_SEL_3" input (at 102.235 50.8 180)
+      (effects (font (size 1.27 1.27)) (justify left))
+    )
+    (pin "CACHE_SEL_2" input (at 102.235 54.61 180)
+      (effects (font (size 1.27 1.27)) (justify left))
+    )
+    (pin "CACHE_SEL_0" input (at 102.235 59.055 180)
+      (effects (font (size 1.27 1.27)) (justify left))
+    )
+    (pin "LOCAL_D[0..7]" bidirectional (at 102.235 79.375 180)
+      (effects (font (size 1.27 1.27)) (justify left))
+    )
+    (pin "LOCAL_A[0..15]" input (at 102.235 75.565 180)
+      (effects (font (size 1.27 1.27)) (justify left))
+    )
+    (instances
+      (project "IOCACHE-128k_ZXspectrum_impl"
+        (path "/532c0392-800e-45cc-8170-6d32f2390e83" (page "2"))
+      )
+    )
+  )
   (sheet_instances
     (path "/" (page "1"))
