File: KiCad7/FujiNet_Z80Bus_Adapters/ZXspectrum_Concept/ZXspectrum_Concept.kicad_sch (KiCad schematic)
At the start: 0 parts

Commit message: KiCad ZXspectrum concept
Connections:
- no-connect marks 0 -> 1
Other:
- sheet SPI ports: added {SPI_INTERNAL}; removed {ESP_SPI_INTERNAL}
Changed lines of the file:
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@@
   (junction (at 204.47 36.83) (diameter 0) (color 0 0 0 0)
   )
+  (junction (at 106.68 73.66) (diameter 0) (color 0 0 0 0)
+  )
   (junction (at 181.61 30.48) (diameter 0) (color 0 0 0 0)
   )
@@
   (junction (at 196.85 43.18) (diameter 0) (color 0 0 0 0)
   )
+  (no_connect (at 109.22 81.28))
   (bus_entry (at 200.66 121.92) (size -2.54 2.54)
     (stroke (width 0) (type default))
@@
     (stroke (width 0) (type default))
   )
+  (wire (pts (xy 86.36 165.1) (xy 106.68 165.1))
+    (stroke (width 0) (type default))
+  )
   (wire (pts (xy 86.36 127) (xy 88.9 127))
     (stroke (width 0) (type default))
@@
     (stroke (width 0) (type default))
   )
+  (wire (pts (xy 109.22 81.28) (xy 111.76 81.28))
+    (stroke (width 0) (type default))
+  )
   (wire (pts (xy 90.17 124.46) (xy 86.36 124.46))
     (stroke (width 0) (type default))
@@
     (stroke (width 0) (type default))
   )
-  (wire (pts (xy 55.88 73.66) (xy 111.76 73.66))
+  (wire (pts (xy 55.88 73.66) (xy 106.68 73.66))
     (stroke (width 0) (type default))
   )
@@
     (stroke (width 0) (type default))
   )
+  (wire (pts (xy 106.68 73.66) (xy 111.76 73.66))
+    (stroke (width 0) (type default))
+  )
+  (wire (pts (xy 106.68 165.1) (xy 106.68 73.66))
+    (stroke (width 0) (type default))
+  )
   (wire (pts (xy 88.9 127) (xy 88.9 162.56))
     (stroke (width 0) (type default))
@@
     (effects (font (size 1.27 1.27)) (justify left bottom))
   )
-  (sheet (at 210.82 53.34) (size 25.4 67.31) (fields_autoplaced)
+  (sheet (at 210.82 52.07) (size 25.4 68.58) (fields_autoplaced)
     (stroke (width 0.1524) (type solid))
     (fill (color 0 0 0 0.0000))
-    (property "Sheetname" "SPI" (at 210.82 52.6284 0)
+    (property "Sheetname" "SPI" (at 210.82 51.3584 0)
       (effects (font (size 1.27 1.27)) (justify left bottom))
     )
@@
       (effects (font (size 1.27 1.27)) (justify left))
     )
-    (pin "{ESP_SPI_INTERNAL}" input (at 210.82 54.61 180)
-      (effects (font (size 1.27 1.27)) (justify left))
-    )
     (pin "{ESP_CONTROL}" output (at 210.82 106.68 180)
+      (effects (font (size 1.27 1.27)) (justify left))
+    )
+    (pin "{SPI_INTERNAL}" input (at 210.82 54.61 180)
       (effects (font (size 1.27 1.27)) (justify left))
     )
@@
     )
   )
-  (sheet (at 210.82 27.94) (size 25.4 21.59) (fields_autoplaced)
+  (sheet (at 210.82 27.94) (size 25.4 20.32) (fields_autoplaced)
     (stroke (width 0.1524) (type solid))
     (fill (color 0 0 0 0.0000))
@@
       (effects (font (size 1.27 1.27)) (justify left bottom))
     )
-    (property "Sheetfile" "../../FujiNet_Z80Bus_Modules/Z80-BUS_ZXspectrum48K/Z80-BUS_ZXspectrum48K.kicad_sch" (at 210.82 50.1146 0)
+    (property "Sheetfile" "../../FujiNet_Z80Bus_Modules/Z80-BUS_ZXspectrum48K/Z80-BUS_ZXspectrum48K.kicad_sch" (at 210.82 48.8446 0)
       (effects (font (size 1.27 1.27)) (justify left top) hide)
     )
