File: KiCad7/FujiNet_Z80Bus_Modules/GLUE_ZXspectrum/GLUE_ZXspectrum_impl/GLUE_ZXspectrum_impl.kicad_sch (KiCad schematic)
At the start: 0 parts

Commit message: GLUE is broken again, logic gate annotation issue
Other:
- added sheet GLUE_ZXspectrum (../GLUE_ZXspectrum.kicad_sch)
Changed lines of the file:
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@@
   )
   (bus_alias "Z80_CONTROL" (members "Z80_CONTROL.RD" "Z80_CONTROL.WR" "Z80_CONTROL.IORQ" "Z80_CONTROL.MEMRQ" "Z80_CONTROL.BUSRQ" "Z80_CONTROL.WAIT" "Z80_CONTROL.ROMCS" "Z80_CONTROL.BUSACK" "Z80_CONTROL.NMI" "Z80_CONTROL.RESET"))
+  (sheet (at 161.29 40.64) (size 62.23 107.95) (fields_autoplaced)
+    (stroke (width 0.1524) (type solid))
+    (fill (color 0 0 0 0.0000))
+    (property "Sheetname" "GLUE_ZXspectrum" (at 161.29 39.9284 0)
+      (effects (font (size 1.27 1.27)) (justify left bottom))
+    )
+    (property "Sheetfile" "../GLUE_ZXspectrum.kicad_sch" (at 161.29 149.1746 0)
+      (effects (font (size 1.27 1.27)) (justify left top))
+    )
+    (pin "WAIT_IO" input (at 161.29 44.45 180)
+      (effects (font (size 1.27 1.27)) (justify left))
+    )
+    (pin "ESP_WAIT_RESET" input (at 161.29 46.99 180)
+      (effects (font (size 1.27 1.27)) (justify left))
+    )
+    (pin "ESP_HARDLOCK" input (at 161.29 49.53 180)
+      (effects (font (size 1.27 1.27)) (justify left))
+    )
+    (pin "Z80_CONTROL.IORQ" input (at 161.29 52.07 180)
+      (effects (font (size 1.27 1.27)) (justify left))
+    )
+    (pin "IORQ_FILTER_BIT" input (at 161.29 54.61 180)
+      (effects (font (size 1.27 1.27)) (justify left))
+    )
+    (pin "PERM_Z80_IORQ" output (at 161.29 57.15 180)
+      (effects (font (size 1.27 1.27)) (justify left))
+    )
+    (pin "Z80_CONTROL.WAIT" input (at 161.29 59.69 180)
+      (effects (font (size 1.27 1.27)) (justify left))
+    )
+    (pin "Z80_HARDLOCK" output (at 161.29 62.23 180)
+      (effects (font (size 1.27 1.27)) (justify left))
+    )
+    (pin "!Z80_HARDLOCK" output (at 161.29 64.77 180)
+      (effects (font (size 1.27 1.27)) (justify left))
+    )
+    (pin "Z80_CONTROL.BUSRQ" input (at 161.29 67.31 180)
+      (effects (font (size 1.27 1.27)) (justify left))
+    )
+    (pin "ESP_CONTROL.MEMRQ" input (at 161.29 69.85 180)
+      (effects (font (size 1.27 1.27)) (justify left))
+    )
+    (pin "CACHE_DATASTATUS" input (at 161.29 72.39 180)
+      (effects (font (size 1.27 1.27)) (justify left))
+    )
+    (pin "Z80_CONTROL.RD" input (at 161.29 74.93 180)
+      (effects (font (size 1.27 1.27)) (justify left))
+    )
+    (pin "ESP_CONTROL.WR" input (at 161.29 77.47 180)
+      (effects (font (size 1.27 1.27)) (justify left))
+    )
+    (pin "Z80_A15" input (at 161.29 80.01 180)
+      (effects (font (size 1.27 1.27)) (justify left))
+    )
+    (pin "Z80_A14" input (at 161.29 82.55 180)
+      (effects (font (size 1.27 1.27)) (justify left))
+    )
+    (pin "ESP_CONTROL.BUSRQ" input (at 161.29 85.09 180)
+      (effects (font (size 1.27 1.27)) (justify left))
+    )
+    (pin "ESP_CONTROL.ROMCS" input (at 161.29 87.63 180)
+      (effects (font (size 1.27 1.27)) (justify left))
+    )
+    (pin "ESP_ROM_WR_PROTECT" input (at 161.29 90.17 180)
+      (effects (font (size 1.27 1.27)) (justify left))
+    )
+    (pin "ESP_CONTROL.IORQ" input (at 161.29 92.71 180)
+      (effects (font (size 1.27 1.27)) (justify left))
+    )
+    (pin "!ESP_HARDLOCK" output (at 161.29 95.25 180)
+      (effects (font (size 1.27 1.27)) (justify left))
+    )
+    (pin "{Z80_BUS_CONTROL}" output (at 161.29 97.79 180)
+      (effects (font (size 1.27 1.27)) (justify left))
+    )
+    (pin "{RIO_CONTROL}" output (at 161.29 100.33 180)
+      (effects (font (size 1.27 1.27)) (justify left))
+    )
+    (pin "{CACHE_CONTROL}" output (at 161.29 102.87 180)
+      (effects (font (size 1.27 1.27)) (justify left))
+    )
+    (pin "ESP_ROMSEL_0" input (at 161.29 105.41 180)
+      (effects (font (size 1.27 1.27)) (justify left))
+    )
+    (pin "ESP_ROMSEL_1" input (at 161.29 107.95 180)
+      (effects (font (size 1.27 1.27)) (justify left))
+    )
+    (pin "Z80_CONTROL.WR" input (at 161.29 110.49 180)
+      (effects (font (size 1.27 1.27)) (justify left))
+    )
+    (pin "Z80_CONTROL.MEMRQ" input (at 161.29 113.03 180)
+      (effects (font (size 1.27 1.27)) (justify left))
+    )
+    (pin "LOCAL_CONTROL.WR" input (at 161.29 115.57 180)
+      (effects (font (size 1.27 1.27)) (justify left))
+    )
+    (pin "LOCAL_CONTROL.IORQ" input (at 161.29 118.11 180)
+      (effects (font (size 1.27 1.27)) (justify left))
+    )
+    (pin "LOCAL_CONTROL.RD" input (at 161.29 120.65 180)
+      (effects (font (size 1.27 1.27)) (justify left))
+    )
+    (pin "LOCAL_CONTROL.MEMRQ" input (at 161.29 123.19 180)
+      (effects (font (size 1.27 1.27)) (justify left))
+    )
+    (pin "Z80_HARDLOCK_RESET" input (at 161.29 125.73 180)
+      (effects (font (size 1.27 1.27)) (justify left))
+    )
+    (pin "Z80_HARDLOCK_SET" input (at 161.29 128.27 180)
+      (effects (font (size 1.27 1.27)) (justify left))
+    )
+    (instances
+      (project "GLUE_ZXspectrum_impl"
+        (path "/532c0392-800e-45cc-8170-6d32f2390e83" (page "2"))
+      )
+    )
+  )
   (sheet_instances
     (path "/" (page "1"))

Commit message: KiCad FIXED GLUE
Parts:
- added IC1: 7404N, Package_DIP:DIP-14_W7.62mm_Socket, symbol 74xx:74HC04
- added IC2, IC5, IC7, IC9: 74HC32N, Package_DIP:DIP-14_W7.62mm_Socket, symbol 74xx:74LS32
- added IC3: 7474N, Package_DIP:DIP-14_W7.62mm_Socket, symbol 74xx:74HC74
- added IC4, IC6, IC? (x3): 74HC08N, Package_DIP:DIP-14_W7.62mm_Socket, symbol 74xx:74LS08
Connections:
- new net +5V: IC1.14 (VCC), IC2.14 (VCC), IC3.14 (VCC), IC4.14 (VCC), IC9.7 (GND)
- new net GND: IC1.7 (GND), IC2.7 (GND), IC3.7 (GND), IC4.7 (GND), IC9.14 (VCC), IC?.4, IC?.4, IC?.5, IC?.5
- no-connect marks 0 -> 2
Other:
- added sheet GLUE_ZXspectrum_connectors (../GLUE_ZXspectrum_connectors.kicad_sch)
- note added: "Unused"

Commit message: Narrow versions of RIO CACHE
Other:
- sheet GLUE_ZXspectrum_connectors: file ../GLUE_ZXspectrum_connectors.kicad_sch -> GLUE_ZXspectrum_connectors.kicad_sch
Changed lines of the file:
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@@
       (effects (font (size 1.27 1.27)) (justify left bottom))
     )
-    (property "Sheetfile" "../GLUE_ZXspectrum_connectors.kicad_sch" (at 196.85 132.6646 0)
+    (property "Sheetfile" "GLUE_ZXspectrum_connectors.kicad_sch" (at 196.85 132.6646 0)
       (effects (font (size 1.27 1.27)) (justify left top))
     )

Commit message: KiCad - Fixed GLUE (need to update concept v2)
Parts:
- removed IC9: 74HC32N, Package_DIP:DIP-14_W7.62mm_Socket, symbol 74xx:74LS32
- added IC?: 74HC08N, Package_DIP:DIP-14_W7.62mm_Socket, symbol 74xx:74LS08
Changed lines of the file:
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@@
+    (stroke (width 0) (type default))
+  )
+  (wire (pts (xy 135.89 160.02) (xy 135.89 161.29))
     (stroke (width 0) (type default))
   )
@@
   )
   (wire (pts (xy 170.18 48.26) (xy 196.85 48.26))
-    (stroke (width 0) (type default))
-  )
-  (wire (pts (xy 135.89 160.02) (xy 135.89 161.29))
     (stroke (width 0) (type default))
   )
@@
         (path "/532c0392-800e-45cc-8170-6d32f2390e83"
           (reference "#PWR05") (unit 1)
+        )
+      )
+    )
+  )
+  (symbol (lib_id "74xx:74LS08") (at 135.89 173.99 0) (unit 2)
+    (in_bom yes) (on_board yes) (dnp no)
+    (property "Reference" "IC?" (at 138.43 170.18 0)
+      (effects (font (size 1.4986 1.4986)) (justify left bottom))
+    )
+    (property "Value" "74HC08N" (at 138.43 179.07 0)
+      (effects (font (size 1.4986 1.4986)) (justify left bottom) hide)
+    )
+    (property "Footprint" "Package_DIP:DIP-14_W7.62mm_Socket" (at 135.89 173.99 0)
+      (effects (font (size 1.27 1.27)) hide)
+    )
+    (property "Datasheet" "http://www.ti.com/lit/gpn/sn74LS08" (at 135.89 173.99 0)
+      (effects (font (size 1.27 1.27)) hide)
+    )
+    (pin "1")
+    (pin "2")
+    (pin "3")
+    (pin "4")
+    (pin "5")
+    (pin "6")
+    (pin "10")
+    (pin "8")
+    (pin "9")
+    (pin "11")
+    (pin "12")
+    (pin "13")
+    (pin "14")
+    (pin "7")
+    (instances
+      (project "FujiNet_Z80Bus_Basic"
+        (path "/35e54075-8ed7-4bf6-837e-479a97e77d5d/344f9fe5-9c02-46d6-8016-81558291d94c"
+          (reference "IC?") (unit 2)
+        )
+      )
+      (project "GLUE_ZXspectrum_impl"
+        (path "/532c0392-800e-45cc-8170-6d32f2390e83"
+          (reference "IC11") (unit 5)
+        )
+        (path "/532c0392-800e-45cc-8170-6d32f2390e83/0da5b4c6-619f-4cd1-829e-b9ad71c924a4/93c14a9e-4a71-4950-b006-2a9affe18130"
+          (reference "IC?") (unit 2)
+        )
+      )
+      (project "GLUE_ZXspectrum"
+        (path "/648e0b91-567a-4972-a379-57b42123c6d5/93c14a9e-4a71-4950-b006-2a9affe18130"
+          (reference "IC?") (unit 2)
         )
       )
@@
           (reference "IC?") (unit 1)
         )
-      )
-    )
-  )
-  (symbol (lib_id "74xx:74LS32") (at 135.89 173.99 0) (unit 5)
-    (in_bom yes) (on_board yes) (dnp no)
-    (property "Reference" "IC9" (at 133.35 173.99 0)
-      (effects (font (size 1.4986 1.4986)) (justify left bottom))
-    )
-    (property "Value" "74HC32N" (at 138.43 179.07 0)
-      (effects (font (size 1.4986 1.4986)) (justify left bottom) hide)
-    )
-    (property "Footprint" "Package_DIP:DIP-14_W7.62mm_Socket" (at 135.89 173.99 0)
-      (effects (font (size 1.27 1.27)) hide)
-    )
-    (property "Datasheet" "http://www.ti.com/lit/gpn/sn74LS32" (at 135.89 173.99 0)
-      (effects (font (size 1.27 1.27)) hide)
-    )
-    (pin "1")
-    (pin "2")
-    (pin "3")
-    (pin "4")
-    (pin "5")
-    (pin "6")
-    (pin "10")
-    (pin "8")
-    (pin "9")
-    (pin "11")
-    (pin "12")
-    (pin "13")
-    (pin "14")
-    (pin "7")
-    (instances
-      (project "GLUE_ZXspectrum_impl"
-        (path "/532c0392-800e-45cc-8170-6d32f2390e83"
-          (reference "IC9") (unit 5)
-        )
-        (path "/532c0392-800e-45cc-8170-6d32f2390e83/0da5b4c6-619f-4cd1-829e-b9ad71c924a4/6bcd45ec-1810-4278-8058-96e26ec9b5f3"
-          (reference "IC9") (unit 1)
-        )
-      )
-      (project "GLUE_ZXspectrum"
-        (path "/648e0b91-567a-4972-a379-57b42123c6d5/6bcd45ec-1810-4278-8058-96e26ec9b5f3"
-          (reference "IC?") (unit 1)
-        )
-      )
-      (project "Logic_core"
-        (path "/79af7f62-e23a-438d-9c25-2567e5e04fca"
-          (reference "IC?") (unit 1)
-        )
