File: KiCad7/FujiNet_Z80Bus_Modules/Base_Schematics/SPI-Z80-BUS_ZXspectrum_V2/SPI-Z80-BUS_ZXspectrum.kicad_sch (KiCad schematic)
At the start: 13 parts

Commit message: KICAD - Restructure and SPI version2 Draft
Parts:
- removed D14: 1N4148, Diode_THT:D_T-1_P5.08mm_Horizontal, symbol Device:D
- added U1: 74HC04, symbol 74xx:74HC04
Connections:
- net ESP_SPI_INT.SCK: now also U1.1
- new net SPI-Z80-BUS_read/ESP_SPI_INT.SCK: U1.2
Other:
- title: FujiNet Z80Bus reference design -> FujiNet Z80 SPI BUS
- moved on the sheet: D12, D13, D15, D3, D4, D?, ESP_CONTROL.Bias, IC?, IC?D, LOCAL_D.Bias, R?, RN?
