File: KiCad7/Z80Bus_Modules/Base_Schematics/GLUE_ZXspectrum/RIO CONTROL.kicad_sch (KiCad schematic)
At the start: 8 parts, among them IC1 7404N, IC4 74HC08N, IC5 74HC32N, IC6 74HC08N, IC7 74HC32N, U1 74HC244N

Commit message: KICAD: Updates to base achemtics for GLUE
Parts:
- removed IC4: 74HC08N, Package_DIP:DIP-14_W7.62mm_Socket, symbol 74xx:74LS08
- removed IC5: 74HC32N, Package_DIP:DIP-14_W7.62mm_Socket, symbol 74xx:74LS32
- removed unit 1 of IC6
- added IC5 (x3), IC7: 74HC32N, Package_DIP:DIP-14_W7.62mm_Socket, symbol 74xx:74LS32
- added unit 1 of IC6 (x3)
Connections:
- net Z80_RD+ESP_IOD_CONFIG+PERM_Z80_IORQ is gone; now on net PERM_Z80_IORQ: U1.8 (1A3)
- net Z80_WR+ESP_IOD_CONFIG is gone; now on net PERMITTED_RIO_WR: U1.6 (1A2)
- net ESP_CONTROL.BUSRQ: now also IC7.9; no longer IC7.10
- net ESP_CONTROL.ROMCS: now also IC5.10
- net RIO_CONTROL.CE: now also IC6.3
- net Z80_A14: now also IC5.10
- net Z80_A15: now also IC5.9
- net Z80_CONTROL.MEMRQ: now also IC5.10
- net ESP_IOD_CONFIG renamed RIO_IOD_CONFIG
- net RIO_IOD_CONFIG: now also IC6.1, IC6.2
- net ESP_ROM_WR_PROTECT renamed ESP_RIO_PROTECT
- net ESP_RIO_PROTECT: now also IC7.10
- net RIO_CONTROL.A16 renamed RIO_IOD_ACCESS
- net RIO_IOD_ACCESS: now also IC6.2, IC6.3
- net RIO_CONTROL.ROM_RDY renamed RIO_ROM_ACCESS
- net RIO_ROM_ACCESS: now also IC5.8, IC6.1, IC6.1
- net ROM_WR_PROTECT+Z80_WR renamed PERMITTED_RIO_WR
- new net: IC7.10, IC7.8
- new net: IC5.8, IC5.9
- new net RIO_CONTROL.DATA_OE: IC6.3
- new net RIO_IOD_DECODE: IC6.2
- new net Z80_ROM_ACCESS: IC5.8, IC5.9
Other:
- note added: "ESP programming IOD"
- note added: "Host ROM base address"
- note added: "RIO Access conditions"
- note added: "RIO write protection"
- company: (none) -> FujiNet
- title: (none) -> RIO Control Logic
- moved on the sheet: D6, IC1F, IC6B, IC7C, IC7D, RN1, U1
