File: KiCad7/Z80Bus_Adapters/ZXspectrum_Concept_v2/ZXspectrum_Concept_v2.kicad_pro.kicad_pcb (KiCad board)
At the start: 2 copper layers, 200 x 130 mm, 45 parts, among them IC1 7404N, IC2 74HC32N, IC3 7474N, IC4 74HC08N, IC5 74HC32N, IC6 74HC08N, IC7 74HC32N, IC8 74HC08N, IC9 74HC32N, J1 PinHeader_2.54mm, J3 LOCAL_D, J4 ESP_SPI_INT, J5 Z80_CONTROL, J6 ESP_CONTROL, J7 LOCAL_A-L, J8 LOCAL_A-H, U1 74HC244N, U2 FREENOVE_ESP32-WROVER-DEV

Commit message: ThatOldNerds V2 of the concept design.
Parts:
- removed D7, D8: 1N4148, Diode_THT:D_T-1_P5.08mm_Horizontal
- removed DIAG-HOST_SYSTEM_BUS1: DIAG-HOST_SYSTEM_BUS, Connector_PinHeader_2.54mm:PinHeader_1x40_P2.54mm_Vertical
- removed IC9: 74HC32N, Package_DIP:DIP-14_W7.62mm_Socket
- removed R5, R6: 10K, Resistor_THT:R_Axial_DIN0207_L6.3mm_D2.5mm_P10.16mm_Horizontal
- added C3: 0.1uf, Capacitor_THT:C_Disc_D7.5mm_W2.5mm_P5.00mm, F.Cu at (188.2, 33.0)
- added C4: 0.1uf, Capacitor_THT:C_Disc_D7.5mm_W2.5mm_P5.00mm, F.Cu at (235.0, 86.4)
- added C5: 0.1uf, Capacitor_THT:C_Disc_D7.5mm_W2.5mm_P5.00mm, F.Cu at (49.0, 79.0)
- added C6: 0.1uf, Capacitor_THT:C_Disc_D7.5mm_W2.5mm_P5.00mm, F.Cu at (207.0, 86.4)
- added H1: MountingHole, MountingHole:MountingHole_2.2mm_M2, F.Cu at (47.0, 29.0)
- added H2: MountingHole, MountingHole:MountingHole_2.2mm_M2, F.Cu at (237.0, 29.0)
- added H3: MountingHole, MountingHole:MountingHole_2.2mm_M2, F.Cu at (237.0, 149.0)
- added H4: MountingHole, MountingHole:MountingHole_2.2mm_M2, F.Cu at (47.0, 149.0)
- added J10: Conn_01x04, Connector_PinHeader_2.54mm:PinHeader_1x04_P2.54mm_Vertical, F.Cu at (55.9, 147.3)
- added J2: LOCAL_D, Connector_PinHeader_2.54mm:PinHeader_1x08_P2.54mm_Vertical, F.Cu at (54.2, 129.1)
- added U3: 74HC244N, Package_DIP:DIP-20_W7.62mm_Socket, F.Cu at (195.8, 48.0)
- J3: value LOCAL_D -> ESP_SPI_INT
- J4: value ESP_SPI_INT -> ESP_CONTROL
- J6: value ESP_CONTROL -> LOCAL_A-L
- J7: value LOCAL_A-L -> LOCAL_A-H
- J8: value LOCAL_A-H -> DIAG-HOST_SYSTEM_BUS; footprint Connector_PinHeader_2.54mm:PinHeader_1x08_P2.54mm_Vertical -> Connector_PinHeader_2.54mm:PinHeader_1x40_P2.54mm_Vertical
- U1: value 74HC244N -> FREENOVE_ESP32-WROVER-DEV; footprint Package_DIP:DIP-20_W7.62mm_Socket -> esp32-wrover:Controller Daughter Board
- U2: value FREENOVE_ESP32-WROVER-DEV -> 74HC00; footprint esp32-wrover:FREENOVE_ESP32-WROVER-DEV -> Package_DIP:DIP-14_W7.62mm
- moved D4 123.5 mm to (98.0, 105.0), turned to 180 degrees
- moved J8 109.1 mm to (96.5, 28.4), turned to 90 degrees
- moved D3 109.0 mm to (116.8, 105.0), turned to 180 degrees
- moved D5 102.5 mm to (116.8, 98.0), turned to 180 degrees
- moved Z80-LOCAL_DATA1 84.8 mm to (75.2, 64.5), turned to 180 degrees
- moved U1 59.9 mm to (221.5, 116.8), turned to 180 degrees
- moved EX_SPI1 57.1 mm to (193.0, 147.3), turned to -90 degrees
- moved U2 44.9 mm to (177.0, 112.8), turned to 0 degrees
- moved IC4 35.5 mm to (150.9, 52.3)
- moved C2 24.7 mm to (159.4, 149.0)
- moved C1 24.6 mm to (117.4, 149.0)
- moved R3 24.6 mm to (137.2, 144.0)
- moved R4 24.6 mm to (141.2, 144.0)
- moved R2 17.5 mm to (203.2, 147.3), turned to 0 degrees
- moved Z80_ADDRLOW1 17.0 mm to (103.1, 64.5), turned to 180 degrees
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Connections:
- net /CACHE connector/CACHE_CONTROL.DATASTATUS+PERM_Z80_IORQ renamed /CACHE_CONTROL.DATASTATUS+PERM_Z80_IORQ
- net /CACHE connector/CACHE_SEL_0 renamed /CACHE_SEL_0
- net /CACHE connector/CACHE_SEL_1 renamed /CACHE_SEL_1
- net /CACHE connector/CACHE_SEL_2 renamed /CACHE_SEL_2
- net /CACHE connector/CACHE_SEL_3 renamed /CACHE_SEL_3
- net /CORE/ESP_SPI_INT.MR renamed /ESP_CONTROL.NMI
- net /GLUE/!ESP_HARDLOCK renamed /~{ESP_HARDLOCK}
- net /GLUE/!Z80_HARDLOCK renamed /Glue Logic/~{Z80_HARDLOCK}
- net /GLUE/CLR_Z80_HARDLOCK renamed /Glue Logic/CLR_Z80_HARDLOCK
- net /GLUE/WAIT_IO renamed /WAIT_IO
- net /GLUE/Z80_HARDLOCK_SET renamed /Z80_HARDLOCK_SET
- C1 pad 1: Net-(C1-Pad1) -> /ESP_WAIT_RESET
- C2 pad 1: /CORE/ESP_WAIT_RESET -> Net-(C2-Pad1)
- CACHE1 pad 1: /CACHE connector/LOCAL_D0 -> /LOCAL_D0
- CACHE1 pad 10: /CACHE connector/LOCAL_A1 -> /LOCAL_A1
- CACHE1 pad 11: /CACHE connector/LOCAL_A2 -> /LOCAL_A2
- CACHE1 pad 12: /CACHE connector/LOCAL_A3 -> /LOCAL_A3
- CACHE1 pad 13: /CACHE connector/LOCAL_A4 -> /LOCAL_A4
- CACHE1 pad 14: /CACHE connector/LOCAL_A5 -> /LOCAL_A5
- CACHE1 pad 15: /CACHE connector/LOCAL_A6 -> /LOCAL_A6
- CACHE1 pad 16: /CACHE connector/LOCAL_A7 -> /LOCAL_A7
- CACHE1 pad 17: /CACHE connector/LOCAL_A8 -> /LOCAL_A8
- CACHE1 pad 18: /CACHE connector/LOCAL_A9 -> /LOCAL_A9
- CACHE1 pad 19: /CACHE connector/LOCAL_A10 -> /LOCAL_A10
- CACHE1 pad 2: /CACHE connector/LOCAL_D1 -> /LOCAL_D1
- CACHE1 pad 20: /CACHE connector/LOCAL_A11 -> /LOCAL_A11
- CACHE1 pad 21: /CACHE connector/LOCAL_A12 -> /LOCAL_A12
- CACHE1 pad 22: /CACHE connector/LOCAL_A13 -> /LOCAL_A13
- CACHE1 pad 23: /CACHE connector/LOCAL_A14 -> /LOCAL_A14
- CACHE1 pad 24: /CACHE connector/LOCAL_A15 -> /LOCAL_A15
- CACHE1 pad 3: /CACHE connector/LOCAL_D2 -> /LOCAL_D2
- CACHE1 pad 4: /CACHE connector/LOCAL_D3 -> /LOCAL_D3
- CACHE1 pad 5: /CACHE connector/LOCAL_D4 -> /LOCAL_D4
- CACHE1 pad 6: /CACHE connector/LOCAL_D5 -> /LOCAL_D5
- CACHE1 pad 7: /CACHE connector/LOCAL_D6 -> /LOCAL_D6
- CACHE1 pad 8: /CACHE connector/LOCAL_D7 -> /LOCAL_D7
- CACHE1 pad 9: /CACHE connector/LOCAL_A0 -> /LOCAL_A0
- CACHE2 pad 12: /CACHE connector/CACHE_DATASTATUS -> /CACHE_DATASTATUS
- CACHE2 pad 2: /CACHE connector/CACHE_CONTROL.A16 -> /CACHE_CONTROL.A16
- CACHE2 pad 3: /CACHE connector/CACHE_CONTROL.WE -> /CACHE_CONTROL.WE
- CACHE2 pad 4: /CACHE connector/CACHE_CONTROL.OE -> /CACHE_CONTROL.OE
- CACHE2 pad 5: /CACHE connector/CACHE_CONTROL.CS -> /CACHE_CONTROL.CS
- CACHE2 pad 7: /CACHE connector/Z80_HARDLOCK -> /Z80_HARDLOCK
- D1 pad 2: /SPI connector/Z80_CONTROL.RESET -> /Z80_CONTROL.RESET
- D2 pad 1: Net-(D2-K) -> /Z80_CONTROL.WAIT
- D2 pad 2: /SPI connector/Z80_CONTROL.WAIT -> /ESP32WRover/ESP_INT
- D3 pad 1: /SPI connector/Z80_CONTROL.WAIT -> /Z80_HARDLOCK_RESET
- D3 pad 2: /CORE/ESP_INT -> /ESP32WRover/ESP_INT
- D4 pad 1: /CORE/Z80_HARDLOCK_RESET -> /Z80_CONTROL.BUSACK
- D4 pad 2: /CORE/ESP_INT -> /ESP32WRover/ESP_INT
- D5 pad 1: /SPI connector/Z80_CONTROL.BUSACK -> Net-(D5-K)
- D5 pad 2: /CORE/ESP_INT -> /Z80_CONTROL.WAIT
- EX_SPI1 pad 1: /CORE/EX_SS -> /ESP32WRover/EX_SS
- EX_SPI1 pad 2: /CORE/EX_SCK -> /ESP32WRover/EX_SCK
- EX_SPI1 pad 3: /CORE/EX_MISO -> /ESP32WRover/EX_MISO
- EX_SPI1 pad 4: /CORE/EX_MOSI -> /ESP32WRover/EX_MOSI
- IC1 pad 1: /CORE/ESP_HARDLOCK -> /ESP_HARDLOCK
- IC1 pad 10: /GLUE/Z80 BUS CONTROL/!CACHE_DATASTATUS -> Net-(IC1-Pad10)
- IC1 pad 11: /CACHE connector/CACHE_DATASTATUS -> /CACHE_DATASTATUS
- IC1 pad 12: Net-(IC1-Pad12) -> /Z80_CONTROL.ROMCS
- IC1 pad 13: Net-(IC1-Pad13) -> /ESP_CONTROL.ROMCS
- IC1 pad 14: +5V -> GND
- IC1 pad 4: Net-(IC1-Pad4) -> /Glue Logic/PRE_Z80_HARDLOCK
- IC1 pad 5: /CORE/Z80_HARDLOCK_RESET -> /Z80_HARDLOCK_RESET
- IC1 pad 7: GND -> unconnected-(IC1G-GND-Pad7)
- IC2 pad 1: Net-(IC1-Pad4) -> /ESP_CONTROL.BUSRQ
- IC2 pad 10: /SPI connector/Z80_CONTROL.IORQ -> /Z80_CONTROL.IORQ
- IC2 pad 11: /GLUE/PERM_Z80_IORQ -> /Glue Logic/RIO_IOD_DECODE
- IC2 pad 12: /RIO connector/Z80_A0 -> /IORQ_FILTER_BITS
- IC2 pad 14: +5V -> unconnected-(IC2E-VCC-Pad14)
- IC2 pad 2: /CORE/ESP_HARDLOCK -> /Z80_CONTROL.BUSACK
- IC2 pad 3: /GLUE/PRE_Z80_HARDLOCK -> /Z80_BUS_CONTROL.Z80_ADD_DIR
- IC2 pad 4: /GLUE/PERM_Z80_IORQ -> /PERM_Z80_IORQ
- IC2 pad 5: /CACHE connector/CACHE_DATASTATUS -> /CACHE_DATASTATUS
- IC2 pad 9: /CORE/ESP_HARDLOCK -> /ESP_HARDLOCK
- IC3 pad 13: /CORE/ESP_WAIT_RESET -> /ESP_WAIT_RESET
- IC3 pad 4: /GLUE/PRE_Z80_HARDLOCK -> /Glue Logic/PRE_Z80_HARDLOCK
- IC3 pad 5: /CACHE connector/Z80_HARDLOCK -> /Z80_HARDLOCK
- IC3 pad 8: Net-(D2-K) -> Net-(D5-K)
- IC4 pad 1: Net-(C1-Pad1) -> Net-(C2-Pad1)
- IC4 pad 10: /GLUE/RIO_CONTROL.A16 -> /LOCAL_CONTROL.RD
- IC4 pad 11: Net-(IC4-Pad11) -> /CACHE_CONTROL.CS
- IC4 pad 12: /GLUE/ESP_IOD_CONFIG -> /PERM_Z80_IORQ
- IC4 pad 13: /GLUE/RIO_CONTROL.ROM_RDY -> /LOCAL_CONTROL.MEMRQ
- IC4 pad 14: +5V -> unconnected-(IC4E-VCC-Pad14)
- IC4 pad 4: /GLUE/PERM_Z80_IORQ -> /ESP_CONTROL.MEMRQ
- IC4 pad 5: /GLUE/ESP_IOD_CONFIG -> /ESP_CONTROL.IORQ
- IC4 pad 6: /GLUE/RIO_CONTROL.A16 -> Net-(IC4-Pad6)
- IC4 pad 7: GND -> unconnected-(IC4E-GND-Pad7)
- IC4 pad 8: /GLUE/RIO_CONTROL.CE -> /CACHE_CONTROL.OE
- IC4 pad 9: Net-(IC4-Pad11) -> /Z80_CONTROL.RD
- IC5 pad 1: /GLUE/ESP_IOD_CONFIG -> /Glue Logic/RIO_IOD_DECODE
- IC5 pad 10: /SPI connector/Z80_CONTROL.MEMRQ -> /LOCAL_A15
- IC5 pad 11: Net-(IC5-Pad11) -> /Glue Logic/RIO CONTROL/PERMITTED_RIO_WR
- IC5 pad 12: /SPI connector/Z80_CONTROL.RD -> /Z80_CONTROL.WR
- IC5 pad 13: /GLUE/ESP_IOD_CONFIG -> /ESP_RIO_PROTECT
- IC5 pad 14: +5V -> unconnected-(IC5E-VCC-Pad14)
- IC5 pad 2: /SPI connector/Z80_CONTROL.WR -> Net-(IC1-Pad10)
- IC5 pad 3: /GLUE/RIO CONTROL/Z80_WR+ESP_IOD_CONFIG -> Net-(IC5-Pad3)
- IC5 pad 4: /SPI connector/ESP_CONTROL.WR -> /Glue Logic/RIO CONTROL/Z80_ROM_ACCESS
- IC5 pad 5: /GLUE/Z80 BUS CONTROL/Z80_DATA_CONNECT -> /ESP_CONTROL.ROMCS
- IC5 pad 6: Net-(IC5-Pad6) -> /RIO_CONTROL.A16
- IC5 pad 7: GND -> unconnected-(IC5E-GND-Pad7)
- IC5 pad 8: /GLUE/RIO_CONTROL.ROM_RDY -> Net-(IC5-Pad8)
- IC5 pad 9: /SPI connector/ESP_CONTROL.ROMCS -> /LOCAL_A14
- IC6 pad 1: /GLUE/PERM_Z80_IORQ -> /Glue Logic/RIO CONTROL/RIO_IOD_CONFIG
- IC6 pad 10: GND -> Net-(IC6-Pad10)
- IC6 pad 11: unconnected-(IC6-Pad11) -> /CACHE_CONTROL.A16
- IC6 pad 12: GND -> /CACHE_DATASTATUS
- IC6 pad 13: GND -> /LOCAL_CONTROL.IORQ
- IC6 pad 2: Net-(IC5-Pad11) -> /Glue Logic/RIO_IOD_DECODE
- IC6 pad 3: /GLUE/RIO CONTROL/Z80_RD+ESP_IOD_CONFIG+PERM_Z80_IORQ -> /Glue Logic/RIO CONTROL/RIO_IOD_ACCESS
- IC6 pad 4: /SPI connector/ESP_CONTROL.MEMRQ -> /Z80_CONTROL.WR
- IC6 pad 5: /SPI connector/ESP_CONTROL.IORQ -> /LOCAL_CONTROL.WR
- IC6 pad 6: Net-(IC1-Pad13) -> /CACHE_CONTROL.WE
- IC6 pad 8: unconnected-(IC6-Pad8) -> /Z80_BUS_CONTROL.Z80_DATA_DIR
- IC6 pad 9: GND -> /ESP_CONTROL.WR
- IC7 pad 1: /GLUE/PERM_Z80_IORQ -> /Glue Logic/RIO_IOD_DECODE
- IC7 pad 10: /SPI connector/ESP_CONTROL.BUSRQ -> /Z80_CONTROL.MEMRQ
- IC7 pad 11: /GLUE/RIO CONTROL/ROM_WR_PROTECT+Z80_WR -> /Z80_BUS_CONTROL.Z80_DATA_OE
- IC7 pad 12: /SPI connector/Z80_CONTROL.WR -> /Z80_BUS_CONTROL.Z80_ADD_DIR
- IC7 pad 13: /CORE/ESP_ROM_WR_PROTECT -> /Glue Logic/RIO_IOD_DECODE
- IC7 pad 14: +5V -> GND
- IC7 pad 2: /GLUE/Z80 BUS CONTROL/!CACHE_DATASTATUS -> /Z80_CONTROL.RD
- IC7 pad 3: Net-(IC7-Pad3) -> Net-(IC6-Pad10)
- IC7 pad 4: /GLUE/Z80 BUS CONTROL/Z80_DATA_CONNECT -> /ESP_CONTROL.BUSRQ
- IC7 pad 5: /GLUE/PERM_Z80_IORQ -> /ESP_RIO_PROTECT
- IC7 pad 6: /GLUE/Z80_BUS_CONTROL.Z80_DATA_OE -> Net-(IC7-Pad6)
- IC7 pad 7: GND -> unconnected-(IC7E-GND-Pad7)
- IC7 pad 8: /GLUE/ESP_IOD_CONFIG -> /Glue Logic/RIO CONTROL/Z80_ROM_ACCESS
- IC7 pad 9: Net-(IC1-Pad12) -> Net-(IC5-Pad8)
- IC8 pad 1: /CACHE connector/CACHE_DATASTATUS -> /RIO_CONTROL.A16
- IC8 pad 10: /SPI connector/LOCAL_CONTROL.RD -> /Z80_BUS_CONTROL.Z80_ADD_DIR
- IC8 pad 11: /CACHE connector/CACHE_CONTROL.CS -> unconnected-(IC8-Pad11)
- IC8 pad 12: /GLUE/PERM_Z80_IORQ -> GND
- IC8 pad 13: /SPI connector/LOCAL_CONTROL.MEMRQ -> GND
- IC8 pad 2: /SPI connector/LOCAL_CONTROL.IORQ -> /Glue Logic/RIO CONTROL/RIO_IOD_CONFIG
- IC8 pad 3: /CACHE connector/CACHE_CONTROL.A16 -> /RIO_CONTROL.DATA_OE
- IC8 pad 4: /SPI connector/Z80_CONTROL.WR -> /RIO_CONTROL.A16
- IC8 pad 5: /SPI connector/LOCAL_CONTROL.WR -> /Glue Logic/RIO CONTROL/RIO_IOD_ACCESS
- IC8 pad 6: /CACHE connector/CACHE_CONTROL.WE -> /RIO_CONTROL.CE
- IC8 pad 8: /CACHE connector/CACHE_CONTROL.OE -> /Z80_BUS_CONTROL.Z80_ADD_OE
- IC8 pad 9: /SPI connector/Z80_CONTROL.RD -> Net-(IC5-Pad3)
- J1 pad 2: /CORE/ESP_PULSE -> /ESP PULSE
- J3 pad 1: /CACHE connector/LOCAL_D0 -> /ESP_SPI_INT.MOSI
- J3 pad 2: /CACHE connector/LOCAL_D1 -> /ESP_SPI_INT.MISO
- J3 pad 3: /CACHE connector/LOCAL_D2 -> /ESP_SPI_INT.SCK
- J3 pad 4: /CACHE connector/LOCAL_D3 -> /ESP_SPI_INT.STC
- J3 pad 5: /CACHE connector/LOCAL_D4 -> /ESP_SPI_INT.PL
- J3 pad 6: /CACHE connector/LOCAL_D5 -> /ESP_SPI_INT.CE
- J3 pad 7: /CACHE connector/LOCAL_D6 -> /ESP_SPI_INT.OE
- J3 pad 8: /CACHE connector/LOCAL_D7 -> /ESP_SPI_INT.MR
- J4 pad 1: /CORE/ESP_SPI_INT.MOSI -> /ESP_CONTROL.RD
- J4 pad 2: /CORE/ESP_SPI_INT.MISO -> /ESP_CONTROL.WR
- J4 pad 3: /CORE/ESP_SPI_INT.SCK -> /ESP_CONTROL.IORQ
- J4 pad 4: /CORE/ESP_SPI_INT.STC -> /ESP_CONTROL.MEMRQ
- J4 pad 5: /CORE/ESP_SPI_INT.PL -> /ESP_CONTROL.BUSRQ
- J4 pad 6: /CORE/ESP_SPI_INT.CE -> /ESP_CONTROL.WAIT
- J4 pad 7: /CORE/ESP_SPI_INT.OE -> /ESP_CONTROL.ROMCS
- J5 pad 1: /SPI connector/Z80_CONTROL.RD -> /Z80_CONTROL.RD
- J5 pad 10: /SPI connector/Z80_CONTROL.RESET -> /Z80_CONTROL.RESET
- J5 pad 2: /SPI connector/Z80_CONTROL.WR -> /Z80_CONTROL.WR
- J5 pad 3: /SPI connector/Z80_CONTROL.IORQ -> /Z80_CONTROL.IORQ
- J5 pad 4: /SPI connector/Z80_CONTROL.MEMRQ -> /Z80_CONTROL.MEMRQ
- J5 pad 5: /SPI connector/Z80_CONTROL.BUSRQ -> /Z80_CONTROL.BUSRQ
- J5 pad 6: /SPI connector/Z80_CONTROL.WAIT -> /Z80_CONTROL.WAIT
- J5 pad 7: /SPI connector/Z80_CONTROL.ROMCS -> /Z80_CONTROL.ROMCS
- J5 pad 8: /SPI connector/Z80_CONTROL.BUSACK -> /Z80_CONTROL.BUSACK
- J5 pad 9: /SPI connector/Z80_CONTROL.NMI -> /Z80_CONTROL.NMI
- J6 pad 1: /SPI connector/ESP_CONTROL.RD -> /LOCAL_A0
- J6 pad 2: /SPI connector/ESP_CONTROL.WR -> /LOCAL_A1
- J6 pad 3: /SPI connector/ESP_CONTROL.IORQ -> /LOCAL_A2
- J6 pad 4: /SPI connector/ESP_CONTROL.MEMRQ -> /LOCAL_A3
- J6 pad 5: /SPI connector/ESP_CONTROL.BUSRQ -> /LOCAL_A4
- J6 pad 6: /SPI connector/ESP_CONTROL.WAIT -> /LOCAL_A5
- J6 pad 7: /SPI connector/ESP_CONTROL.ROMCS -> /LOCAL_A6
- J6 pad 8: /SPI connector/ESP_CONTROL.NMI -> /LOCAL_A7
- J7 pad 1: /CACHE connector/LOCAL_A0 -> /LOCAL_A8
- J7 pad 2: /CACHE connector/LOCAL_A1 -> /LOCAL_A9
- J7 pad 3: /CACHE connector/LOCAL_A2 -> /LOCAL_A10
- J7 pad 4: /CACHE connector/LOCAL_A3 -> /LOCAL_A11
- J7 pad 5: /CACHE connector/LOCAL_A4 -> /LOCAL_A12
- J7 pad 6: /CACHE connector/LOCAL_A5 -> /LOCAL_A13
- J7 pad 7: /CACHE connector/LOCAL_A6 -> /LOCAL_A14
- J7 pad 8: /CACHE connector/LOCAL_A7 -> /LOCAL_A15
- J8 pad 1: /CACHE connector/LOCAL_A8 -> /Z80_CONTROL.RD
- J8 pad 2: /CACHE connector/LOCAL_A9 -> /Z80_CONTROL.WR
- J8 pad 3: /CACHE connector/LOCAL_A10 -> /Z80_CONTROL.IORQ
- J8 pad 4: /CACHE connector/LOCAL_A11 -> /Z80_CONTROL.MEMRQ
- J8 pad 5: /CACHE connector/LOCAL_A12 -> /Z80_CONTROL.BUSRQ
- J8 pad 6: /CACHE connector/LOCAL_A13 -> /Z80_CONTROL.WAIT
- J8 pad 7: /CACHE connector/LOCAL_A14 -> /Z80_CONTROL.NMI
- J8 pad 8: /CACHE connector/LOCAL_A15 -> /Z80_CONTROL.ROMCS
- LOCAL_CONTROL1 pad 1: /SPI connector/LOCAL_CONTROL.RD -> /LOCAL_CONTROL.RD
- LOCAL_CONTROL1 pad 2: /SPI connector/LOCAL_CONTROL.WR -> /LOCAL_CONTROL.WR
- LOCAL_CONTROL1 pad 3: /SPI connector/LOCAL_CONTROL.IORQ -> /LOCAL_CONTROL.IORQ
- LOCAL_CONTROL1 pad 4: /SPI connector/LOCAL_CONTROL.MEMRQ -> /LOCAL_CONTROL.MEMRQ
- R1 pad 1: /CORE/ESP_INT -> /ESP32WRover/ESP_INT
- R2 pad 2: /CORE/ESP_INT -> /ESP32WRover/ESP_INT
- R3 pad 2: Net-(C1-Pad1) -> Net-(C2-Pad1)
- R4 pad 2: /CORE/ESP_WAIT_RESET -> /ESP_WAIT_RESET
- RIO1 pad 1: /RIO connector/Z80_D0 -> /Z80_D0
- RIO1 pad 10: /RIO connector/Z80_A1 -> /Z80_A1
- RIO1 pad 11: /RIO connector/Z80_A2 -> /Z80_A2
- RIO1 pad 12: /RIO connector/Z80_A3 -> /Z80_A3
- RIO1 pad 13: /RIO connector/Z80_A4 -> /Z80_A4
- RIO1 pad 14: /RIO connector/Z80_A5 -> /Z80_A5
- RIO1 pad 15: /RIO connector/Z80_A6 -> /Z80_A6
- RIO1 pad 16: /RIO connector/Z80_A7 -> /Z80_A7
- RIO1 pad 17: /RIO connector/Z80_A8 -> /Z80_A8
- RIO1 pad 18: /RIO connector/Z80_A9 -> /Z80_A9
- RIO1 pad 19: /RIO connector/Z80_A10 -> /Z80_A10
- RIO1 pad 2: /RIO connector/Z80_D1 -> /Z80_D1
- RIO1 pad 20: /RIO connector/Z80_A11 -> /Z80_A11
- RIO1 pad 21: /RIO connector/Z80_A12 -> /Z80_A12
- RIO1 pad 22: /RIO connector/Z80_A13 -> /Z80_A13
- RIO1 pad 23: /RIO connector/Z80_A14 -> /Z80_A14
- RIO1 pad 24: /RIO connector/Z80_A15 -> /Z80_A15
- RIO1 pad 3: /RIO connector/Z80_D2 -> /Z80_D2
- RIO1 pad 4: /RIO connector/Z80_D3 -> /Z80_D3
- RIO1 pad 5: /RIO connector/Z80_D4 -> /Z80_D4
- RIO1 pad 6: /RIO connector/Z80_D5 -> /Z80_D5
- RIO1 pad 7: /RIO connector/Z80_D6 -> /Z80_D6
- RIO1 pad 8: /RIO connector/Z80_D7 -> /Z80_D7
- RIO1 pad 9: /RIO connector/Z80_A0 -> /Z80_A0
- RIO2 pad 13: /CACHE connector/CACHE_DATASTATUS -> /CACHE_DATASTATUS
- RIO2 pad 15: /CORE/Z80_HARDLOCK_RESET -> /Z80_HARDLOCK_RESET
- RIO2 pad 17: /GLUE/PERM_Z80_IORQ -> /PERM_Z80_IORQ
- RIO2 pad 2: /GLUE/RIO_CONTROL.A16 -> /RIO_CONTROL.A16
- RIO2 pad 3: /GLUE/RIO_CONTROL.A15 -> /RIO_CONTROL.A15
- RIO2 pad 4: /GLUE/RIO_CONTROL.A14 -> /RIO_CONTROL.A14
- RIO2 pad 5: /GLUE/RIO_CONTROL.WE -> /RIO_CONTROL.WE
- RIO2 pad 6: /GLUE/RIO_CONTROL.CE -> /RIO_CONTROL.CE
- RIO2 pad 7: /GLUE/RIO_CONTROL.OE -> /RIO_CONTROL.OE
- RIO2 pad 8: /GLUE/RIO_CONTROL.ROM_RDY -> /RIO_CONTROL.DATA_OE
- RN1 pad 2: /GLUE/RIO_CONTROL.A14 -> /RIO_CONTROL.A14
- RN1 pad 3: /GLUE/RIO_CONTROL.A15 -> /RIO_CONTROL.A15
- RN1 pad 4: /GLUE/RIO_CONTROL.WE -> /RIO_CONTROL.WE
- RN1 pad 5: /GLUE/RIO_CONTROL.OE -> /RIO_CONTROL.OE
- U1 pad 1: /GLUE/RIO_CONTROL.A16 -> unconnected-(U1-3V3-Pad1)
- U1 pad 10: GND -> /ESP_SPI_INT.STC
- U1 pad 11: /SPI connector/Z80_CONTROL.RD -> /ESP PULSE
- U1 pad 12: /GLUE/RIO_CONTROL.OE -> /ESP32WRover/EX_SCK
- U1 pad 13: /GLUE/RIO CONTROL/ROM_WR_PROTECT+Z80_WR -> /ESP32WRover/EX_MISO
- U1 pad 14: /GLUE/RIO_CONTROL.WE -> unconnected-(U1-GND-Pad14)
- U1 pad 15: /CORE/ESP_ROMSEL_0 -> /ESP32WRover/EX_MOSI
- U1 pad 16: /GLUE/RIO_CONTROL.A15 -> unconnected-(U1-GPIO9-Pad16)
- U1 pad 17: /CORE/ESP_ROMSEL_1 -> unconnected-(U1-GPIO10-Pad17)
- U1 pad 18: /GLUE/RIO_CONTROL.A14 -> /ESP_WAIT_RESET
- U1 pad 19: /GLUE/RIO_CONTROL.ROM_RDY -> unconnected-(U1-+5v-Pad19)
- U1 pad 2: /RIO connector/Z80_A15 -> unconnected-(U1-EN-Pad2)
- U1 pad 3: /GLUE/RIO_CONTROL.A14 -> /ESP32WRover/ESP_INT
- U1 pad 4: /RIO connector/Z80_A14 -> /Z80_HARDLOCK
- U1 pad 5: /GLUE/RIO_CONTROL.A15 -> unconnected-(U1-GPIO34-Pad5)
- U1 pad 6: /GLUE/RIO CONTROL/Z80_WR+ESP_IOD_CONFIG -> unconnected-(U1-GPIO35-Pad6)
- U1 pad 7: /GLUE/RIO_CONTROL.WE -> unconnected-(U1-GPIO32-Pad7)
- U1 pad 8: /GLUE/RIO CONTROL/Z80_RD+ESP_IOD_CONFIG+PERM_Z80_IORQ -> /ESP_SPI_INT.OE
- U1 pad 9: /GLUE/RIO_CONTROL.OE -> /ESP_SPI_INT.PL
- U2 pad 1: unconnected-(U2-3V3-Pad1) -> Net-(IC4-Pad6)
- U2 pad 10: /CORE/ESP_SPI_INT.STC -> Net-(U2-Pad10)
- U2 pad 11: /CORE/ESP_PULSE -> unconnected-(U2-Pad11)
- U2 pad 12: /CORE/EX_SCK -> GND
- U2 pad 13: /CORE/EX_MISO -> GND
- U2 pad 14: unconnected-(U2-GND-Pad14) -> +5V
- U2 pad 2: unconnected-(U2-EN-Pad2) -> Net-(IC4-Pad6)
- U2 pad 3: /CORE/ESP_INT -> Net-(U2-Pad3)
- U2 pad 4: /CACHE connector/Z80_HARDLOCK -> Net-(U2-Pad3)
- U2 pad 5: unconnected-(U2-GPIO34-Pad5) -> Net-(IC7-Pad6)
- U2 pad 6: unconnected-(U2-GPIO35-Pad6) -> Net-(U2-Pad10)
- U2 pad 7: unconnected-(U2-GPIO32-Pad7) -> GND
- U2 pad 8: /CORE/ESP_SPI_INT.OE -> /Glue Logic/RIO CONTROL/RIO_IOD_CONFIG
- U2 pad 9: /CORE/ESP_SPI_INT.PL -> Net-(U2-Pad10)
- Z80-LOCAL_DATA1 pad 1: /GLUE/Z80_BUS_CONTROL.Z80_DATA_DIR -> /Z80_BUS_CONTROL.Z80_DATA_DIR
- Z80-LOCAL_DATA1 pad 11: /CACHE connector/LOCAL_D7 -> /LOCAL_D7
- Z80-LOCAL_DATA1 pad 12: /CACHE connector/LOCAL_D6 -> /LOCAL_D6
- Z80-LOCAL_DATA1 pad 13: /CACHE connector/LOCAL_D5 -> /LOCAL_D5
- Z80-LOCAL_DATA1 pad 14: /CACHE connector/LOCAL_D4 -> /LOCAL_D4
- Z80-LOCAL_DATA1 pad 15: /CACHE connector/LOCAL_D3 -> /LOCAL_D3
- Z80-LOCAL_DATA1 pad 16: /CACHE connector/LOCAL_D2 -> /LOCAL_D2
- Z80-LOCAL_DATA1 pad 17: /CACHE connector/LOCAL_D1 -> /LOCAL_D1
- Z80-LOCAL_DATA1 pad 18: /CACHE connector/LOCAL_D0 -> /LOCAL_D0
- Z80-LOCAL_DATA1 pad 19: /GLUE/Z80_BUS_CONTROL.Z80_DATA_OE -> /Z80_BUS_CONTROL.Z80_DATA_OE
- Z80-LOCAL_DATA1 pad 2: /RIO connector/Z80_D0 -> /Z80_D0
- Z80-LOCAL_DATA1 pad 3: /RIO connector/Z80_D1 -> /Z80_D1
- Z80-LOCAL_DATA1 pad 4: /RIO connector/Z80_D2 -> /Z80_D2
- Z80-LOCAL_DATA1 pad 5: /RIO connector/Z80_D3 -> /Z80_D3
- Z80-LOCAL_DATA1 pad 6: /RIO connector/Z80_D4 -> /Z80_D4
- Z80-LOCAL_DATA1 pad 7: /RIO connector/Z80_D5 -> /Z80_D5
- Z80-LOCAL_DATA1 pad 8: /RIO connector/Z80_D6 -> /Z80_D6
- Z80-LOCAL_DATA1 pad 9: /RIO connector/Z80_D7 -> /Z80_D7
- Z80_ADDRHIGH1 pad 1: /GLUE/Z80_BUS_CONTROL.Z80_ADD_DIR -> /Z80_BUS_CONTROL.Z80_ADD_DIR
- Z80_ADDRHIGH1 pad 11: /CACHE connector/LOCAL_A15 -> /LOCAL_A15
- Z80_ADDRHIGH1 pad 12: /CACHE connector/LOCAL_A14 -> /LOCAL_A14
- Z80_ADDRHIGH1 pad 13: /CACHE connector/LOCAL_A13 -> /LOCAL_A13
- Z80_ADDRHIGH1 pad 14: /CACHE connector/LOCAL_A12 -> /LOCAL_A12
- Z80_ADDRHIGH1 pad 15: /CACHE connector/LOCAL_A11 -> /LOCAL_A11
- Z80_ADDRHIGH1 pad 16: /CACHE connector/LOCAL_A10 -> /LOCAL_A10
- Z80_ADDRHIGH1 pad 17: /CACHE connector/LOCAL_A9 -> /LOCAL_A9
- Z80_ADDRHIGH1 pad 18: /CACHE connector/LOCAL_A8 -> /LOCAL_A8
- Z80_ADDRHIGH1 pad 19: /GLUE/Z80_BUS_CONTROL.Z80_ADD_OE -> /Z80_BUS_CONTROL.Z80_ADD_OE
- Z80_ADDRHIGH1 pad 2: /RIO connector/Z80_A8 -> /Z80_A8
- Z80_ADDRHIGH1 pad 3: /RIO connector/Z80_A9 -> /Z80_A9
- Z80_ADDRHIGH1 pad 4: /RIO connector/Z80_A10 -> /Z80_A10
- Z80_ADDRHIGH1 pad 5: /RIO connector/Z80_A11 -> /Z80_A11
- Z80_ADDRHIGH1 pad 6: /RIO connector/Z80_A12 -> /Z80_A12
- Z80_ADDRHIGH1 pad 7: /RIO connector/Z80_A13 -> /Z80_A13
- Z80_ADDRHIGH1 pad 8: /RIO connector/Z80_A14 -> /Z80_A14
- Z80_ADDRHIGH1 pad 9: /RIO connector/Z80_A15 -> /Z80_A15
- Z80_ADDRLOW1 pad 1: /GLUE/Z80_BUS_CONTROL.Z80_ADD_DIR -> /Z80_BUS_CONTROL.Z80_ADD_DIR
- Z80_ADDRLOW1 pad 11: /CACHE connector/LOCAL_A7 -> /LOCAL_A7
- Z80_ADDRLOW1 pad 12: /CACHE connector/LOCAL_A6 -> /LOCAL_A6
- Z80_ADDRLOW1 pad 13: /CACHE connector/LOCAL_A5 -> /LOCAL_A5
- Z80_ADDRLOW1 pad 14: /CACHE connector/LOCAL_A4 -> /LOCAL_A4
- Z80_ADDRLOW1 pad 15: /CACHE connector/LOCAL_A3 -> /LOCAL_A3
- Z80_ADDRLOW1 pad 16: /CACHE connector/LOCAL_A2 -> /LOCAL_A2
- Z80_ADDRLOW1 pad 17: /CACHE connector/LOCAL_A1 -> /LOCAL_A1
- Z80_ADDRLOW1 pad 18: /CACHE connector/LOCAL_A0 -> /LOCAL_A0
- Z80_ADDRLOW1 pad 19: /GLUE/Z80_BUS_CONTROL.Z80_ADD_OE -> /Z80_BUS_CONTROL.Z80_ADD_OE
- Z80_ADDRLOW1 pad 2: /RIO connector/Z80_A0 -> /Z80_A0
- Z80_ADDRLOW1 pad 3: /RIO connector/Z80_A1 -> /Z80_A1
- Z80_ADDRLOW1 pad 4: /RIO connector/Z80_A2 -> /Z80_A2
- Z80_ADDRLOW1 pad 5: /RIO connector/Z80_A3 -> /Z80_A3
- Z80_ADDRLOW1 pad 6: /RIO connector/Z80_A4 -> /Z80_A4
- Z80_ADDRLOW1 pad 7: /RIO connector/Z80_A5 -> /Z80_A5
- Z80_ADDRLOW1 pad 8: /RIO connector/Z80_A6 -> /Z80_A6
- Z80_ADDRLOW1 pad 9: /RIO connector/Z80_A7 -> /Z80_A7
Routing:
- net /SPI connector/Z80_CONTROL.BUSACK: track 458.4 -> 0.00 mm, vias 1 -> 0
- net /SPI connector/Z80_CONTROL.WAIT: track 453.3 -> 0.00 mm, vias 2 -> 0
- net /SPI connector/Z80_CONTROL.RD: track 405.4 -> 0.00 mm, vias 7 -> 0
- net /CACHE_DATASTATUS: track 0.00 -> 392.1 mm, vias 0 -> 1
- net /Z80_CONTROL.RESET: track 0.00 -> 391.4 mm, vias 0 -> 4
- net /Z80_CONTROL.WR: track 0.00 -> 384.8 mm, vias 0 -> 3
- net /CACHE connector/CACHE_DATASTATUS: track 361.8 -> 0.00 mm, vias 3 -> 0
- net /Z80_HARDLOCK: track 0.00 -> 298.4 mm, vias 0 -> 2
- net /RIO connector/Z80_A0: track 283.8 -> 0.00 mm, vias 1 -> 0
- net /RIO_CONTROL.A16: track 0.00 -> 281.8 mm, vias 0 -> 1
- net /LOCAL_A14: track 0.00 -> 274.5 mm, vias 0 -> 2
- net /CACHE connector/Z80_HARDLOCK: track 271.6 -> 0.00 mm, vias 4 -> 0
- net /SPI connector/Z80_CONTROL.RESET: track 259.4 -> 0.00 mm, vias 2 -> 0
- net /SPI connector/Z80_CONTROL.BUSRQ: track 253.8 -> 0.00 mm, vias 3 -> 0
- net /Z80_BUS_CONTROL.Z80_ADD_DIR: track 0.00 -> 253.7 mm, vias 0 -> 4
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