File: KiCad7/Z80Bus_Adapters/ZXspectrum_Concept_v2/Impl/IOCACHE-128K_ZXspectrum_impl_narrow_V1/IOCACHE-128K_ZXspectrum_connectors.kicad_sch (KiCad schematic)
At the start: 2 parts

Commit message: ThatOldNerds V2 of the concept design.
Parts:
- renumbered CACHE1 to CACHE?, CACHE2 to CACHE?
Changed lines of the file:
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@@
   (symbol (lib_id "Connector:Conn_01x24_Socket") (at 87.63 138.43 0) (unit 1)
     (in_bom yes) (on_board yes) (dnp no)
-    (property "Reference" "CACHE1" (at 89.535 139.065 0)
+    (property "Reference" "CACHE?" (at 89.535 139.065 0)
       (effects (font (size 1.27 1.27)) (justify left))
     )
@@
       (project "IOCACHE-128K_ZXspectrum_impl_narrow"
         (path "/532c0392-800e-45cc-8170-6d32f2390e83/84439c1e-570e-4c72-8fb1-44f7d27a07e5"
+          (reference "CACHE?") (unit 1)
+        )
+      )
+      (project "ZXspectrum_Concept_v2.kicad_pro"
+        (path "/55b3df09-427f-490b-af7e-cf3fd0c70b9f/c8a8ec74-821c-4c02-bbb4-83fc8ae5c878"
           (reference "CACHE1") (unit 1)
         )
@@
       (project "IOCACHE-128K_ZXspectrum"
         (path "/884c7ad2-5794-4c2b-8afa-8e07fcecd42b/f9303533-0d3f-4609-9fa9-076efff1786c"
-          (reference "J2") (unit 1)
+          (reference "J?") (unit 1)
         )
       )
@@
   (symbol (lib_id "Connector:Conn_01x14_Socket") (at 115.57 106.68 90) (mirror x) (unit 1)
     (in_bom yes) (on_board yes) (dnp no)
-    (property "Reference" "CACHE2" (at 116.205 108.585 0)
+    (property "Reference" "CACHE?" (at 116.205 108.585 0)
       (effects (font (size 1.27 1.27)) (justify left))
     )
@@
       (project "IOCACHE-128K_ZXspectrum_impl_narrow"
         (path "/532c0392-800e-45cc-8170-6d32f2390e83/84439c1e-570e-4c72-8fb1-44f7d27a07e5"
+          (reference "CACHE?") (unit 1)
+        )
+      )
+      (project "ZXspectrum_Concept_v2.kicad_pro"
+        (path "/55b3df09-427f-490b-af7e-cf3fd0c70b9f/c8a8ec74-821c-4c02-bbb4-83fc8ae5c878"
           (reference "CACHE2") (unit 1)
         )
@@
       (project "IOCACHE-128K_ZXspectrum"
         (path "/884c7ad2-5794-4c2b-8afa-8e07fcecd42b/f9303533-0d3f-4609-9fa9-076efff1786c"
-          (reference "J1") (unit 1)
+          (reference "J?") (unit 1)
         )
       )
@@
   (symbol (lib_id "power:GND") (at 137.16 99.06 90) (mirror x) (unit 1)
     (in_bom yes) (on_board yes) (dnp no) (fields_autoplaced)
-    (property "Reference" "#PWR042" (at 143.51 99.06 0)
+    (property "Reference" "#PWR017" (at 143.51 99.06 0)
       (effects (font (size 1.27 1.27)) hide)
     )
@@
     (pin "1")
     (instances
+      (project "ZXspectrum_Concept_v2.kicad_pro"
+        (path "/55b3df09-427f-490b-af7e-cf3fd0c70b9f/c8a8ec74-821c-4c02-bbb4-83fc8ae5c878"
+          (reference "#PWR017") (unit 1)
+        )
+      )
       (project "IOCACHE-128K_ZXspectrum"
         (path "/884c7ad2-5794-4c2b-8afa-8e07fcecd42b/f9303533-0d3f-4609-9fa9-076efff1786c"
-          (reference "#PWR09") (unit 1)
+          (reference "#PWR?") (unit 1)
         )
       )
@@
   (symbol (lib_id "power:+5V") (at 97.79 99.06 90) (mirror x) (unit 1)
     (in_bom yes) (on_board yes) (dnp no) (fields_autoplaced)
-    (property "Reference" "#PWR0108" (at 101.6 99.06 0)
+    (property "Reference" "#PWR016" (at 101.6 99.06 0)
       (effects (font (size 1.27 1.27)) hide)
     )
@@
     (pin "1")
     (instances
+      (project "ZXspectrum_Concept_v2.kicad_pro"
+        (path "/55b3df09-427f-490b-af7e-cf3fd0c70b9f/c8a8ec74-821c-4c02-bbb4-83fc8ae5c878"
+          (reference "#PWR016") (unit 1)
+        )
+      )
       (project "IOCACHE-128K_ZXspectrum"
         (path "/884c7ad2-5794-4c2b-8afa-8e07fcecd42b/f9303533-0d3f-4609-9fa9-076efff1786c"
-          (reference "#PWR08") (unit 1)
+          (reference "#PWR?") (unit 1)
         )
       )
