File: KiCad7/Z80Bus_Adapters/ZXspectrum_Concept_v2/Impl/RIO-128K_ZXspectrum_impl_narrow_V1/RIO-128K_ZXspectrum_connector.kicad_sch (KiCad schematic)
At the start: 2 parts

Commit message: ThatOldNerds V2 of the concept design.
Parts:
- renumbered RIO2 to RIO?, RIO1 to RIO?
Connections:
- net RIO_CONTROL.ROM_RDY renamed RIO_CONTROL.DATA_OE
Changed lines of the file:
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@@
 (kicad_sch (version 20230121) (generator eeschema)
   (paper "A4")
+  (bus_entry (at 62.23 63.5) (size 2.54 2.54)
+    (stroke (width 0) (type default))
+  )
+  (bus_entry (at 64.77 81.28) (size -2.54 -2.54)
+    (stroke (width 0) (type default))
+  )
+  (bus_entry (at 71.12 40.64) (size 2.54 2.54)
+    (stroke (width 0) (type default))
+  )
+  (bus_entry (at 62.23 66.04) (size 2.54 2.54)
+    (stroke (width 0) (type default))
+  )
+  (bus_entry (at 71.12 33.02) (size 2.54 2.54)
+    (stroke (width 0) (type default))
+  )
+  (bus_entry (at 184.15 36.83) (size -2.54 2.54)
+    (stroke (width 0) (type default))
+  )
+  (bus_entry (at 71.12 50.8) (size 2.54 2.54)
+    (stroke (width 0) (type default))
+  )
+  (bus_entry (at 71.12 43.18) (size 2.54 2.54)
+    (stroke (width 0) (type default))
+  )
+  (bus_entry (at 64.77 83.82) (size -2.54 -2.54)
+    (stroke (width 0) (type default))
+  )
+  (bus_entry (at 64.77 78.74) (size -2.54 -2.54)
+    (stroke (width 0) (type default))
+  )
+  (bus_entry (at 62.23 68.58) (size 2.54 2.54)
+    (stroke (width 0) (type default))
+  )
+  (bus_entry (at 71.12 45.72) (size 2.54 2.54)
+    (stroke (width 0) (type default))
+  )
+  (bus_entry (at 62.23 86.36) (size 2.54 2.54)
+    (stroke (width 0) (type default))
+  )
+  (bus_entry (at 62.23 73.66) (size 2.54 2.54)
+    (stroke (width 0) (type default))
+  )
+  (bus_entry (at 71.12 38.1) (size 2.54 2.54)
+    (stroke (width 0) (type default))
+  )
+  (bus_entry (at 62.23 58.42) (size 2.54 2.54)
+    (stroke (width 0) (type default))
+  )
+  (bus_entry (at 184.15 39.37) (size -2.54 2.54)
+    (stroke (width 0) (type default))
+  )
+  (bus_entry (at 184.15 46.99) (size -2.54 2.54)
+    (stroke (width 0) (type default))
+  )
+  (bus_entry (at 62.23 91.44) (size 2.54 2.54)
+    (stroke (width 0) (type default))
+  )
+  (bus_entry (at 62.23 71.12) (size 2.54 2.54)
+    (stroke (width 0) (type default))
+  )
+  (bus_entry (at 184.15 44.45) (size -2.54 2.54)
+    (stroke (width 0) (type default))
+  )
   (bus_entry (at 184.15 49.53) (size -2.54 2.54)
     (stroke (width 0) (type default))
   )
-  (bus_entry (at 62.23 63.5) (size 2.54 2.54)
-    (stroke (width 0) (type default))
-  )
-  (bus_entry (at 64.77 81.28) (size -2.54 -2.54)
-    (stroke (width 0) (type default))
-  )
-  (bus_entry (at 71.12 40.64) (size 2.54 2.54)
-    (stroke (width 0) (type default))
-  )
-  (bus_entry (at 62.23 66.04) (size 2.54 2.54)
-    (stroke (width 0) (type default))
-  )
-  (bus_entry (at 71.12 33.02) (size 2.54 2.54)
-    (stroke (width 0) (type default))
-  )
-  (bus_entry (at 184.15 36.83) (size -2.54 2.54)
-    (stroke (width 0) (type default))
-  )
-  (bus_entry (at 71.12 50.8) (size 2.54 2.54)
-    (stroke (width 0) (type default))
-  )
-  (bus_entry (at 71.12 43.18) (size 2.54 2.54)
-    (stroke (width 0) (type default))
-  )
-  (bus_entry (at 64.77 83.82) (size -2.54 -2.54)
-    (stroke (width 0) (type default))
-  )
-  (bus_entry (at 64.77 78.74) (size -2.54 -2.54)
-    (stroke (width 0) (type default))
-  )
-  (bus_entry (at 62.23 68.58) (size 2.54 2.54)
-    (stroke (width 0) (type default))
-  )
-  (bus_entry (at 71.12 45.72) (size 2.54 2.54)
-    (stroke (width 0) (type default))
-  )
-  (bus_entry (at 62.23 86.36) (size 2.54 2.54)
-    (stroke (width 0) (type default))
-  )
-  (bus_entry (at 62.23 73.66) (size 2.54 2.54)
-    (stroke (width 0) (type default))
-  )
-  (bus_entry (at 71.12 38.1) (size 2.54 2.54)
-    (stroke (width 0) (type default))
-  )
-  (bus_entry (at 62.23 58.42) (size 2.54 2.54)
-    (stroke (width 0) (type default))
-  )
-  (bus_entry (at 184.15 39.37) (size -2.54 2.54)
-    (stroke (width 0) (type default))
-  )
-  (bus_entry (at 184.15 46.99) (size -2.54 2.54)
-    (stroke (width 0) (type default))
-  )
-  (bus_entry (at 62.23 91.44) (size 2.54 2.54)
-    (stroke (width 0) (type default))
-  )
-  (bus_entry (at 62.23 71.12) (size 2.54 2.54)
-    (stroke (width 0) (type default))
-  )
-  (bus_entry (at 184.15 44.45) (size -2.54 2.54)
-    (stroke (width 0) (type default))
-  )
   (bus_entry (at 71.12 35.56) (size 2.54 2.54)
     (stroke (width 0) (type default))
@@
     (stroke (width 0) (type default))
   )
+  (wire (pts (xy 181.61 52.07) (xy 156.21 52.07))
+    (stroke (width 0) (type default))
+  )
   (wire (pts (xy 85.09 38.1) (xy 73.66 38.1))
     (stroke (width 0) (type default))
@@
     (stroke (width 0) (type default))
   )
-  (bus (pts (xy 184.15 49.53) (xy 184.15 50.8))
-    (stroke (width 0) (type default))
-  )
   (wire (pts (xy 156.21 74.93) (xy 163.83 74.93))
     (stroke (width 0) (type default))
@@
     (stroke (width 0) (type default))
   )
-  (wire (pts (xy 156.21 52.07) (xy 181.61 52.07))
-    (stroke (width 0) (type default))
-  )
   (bus (pts (xy 71.12 45.72) (xy 71.12 48.26))
     (stroke (width 0) (type default))
@@
     (effects (font (size 1.27 1.27)) (justify left bottom))
   )
+  (label "RIO_CONTROL.DATA_OE" (at 156.21 52.07 0) (fields_autoplaced)
+    (effects (font (size 1.27 1.27)) (justify left bottom))
+  )
   (label "Z80_D1" (at 73.66 38.1 0) (fields_autoplaced)
     (effects (font (size 1.27 1.27)) (justify left bottom))
@@
   )
   (label "Z80_A11" (at 64.77 83.82 0) (fields_autoplaced)
-    (effects (font (size 1.27 1.27)) (justify left bottom))
-  )
-  (label "RIO_CONTROL.ROM_RDY" (at 156.21 52.07 0) (fields_autoplaced)
     (effects (font (size 1.27 1.27)) (justify left bottom))
   )
@@
   (symbol (lib_id "power:+5V") (at 160.02 30.48 0) (unit 1)
     (in_bom yes) (on_board yes) (dnp no) (fields_autoplaced)
-    (property "Reference" "#PWR0102" (at 160.02 34.29 0)
+    (property "Reference" "#PWR?" (at 160.02 34.29 0)
       (effects (font (size 1.27 1.27)) hide)
     )
@@
       (project "ZXspectrum_Concept_v2.kicad_pro"
         (path "/532c0392-800e-45cc-8170-6d32f2390e83/8f76c5c7-fe36-4f58-b465-2615c9dcfdfb"
-          (reference "#PWR0102") (unit 1)
+          (reference "#PWR?") (unit 1)
+        )
+      )
+      (project "ZXspectrum_Concept_v2.kicad_pro"
+        (path "/55b3df09-427f-490b-af7e-cf3fd0c70b9f/0d5f1905-044f-4186-8c0e-e74aa689b436"
+          (reference "#PWR018") (unit 1)
         )
       )
       (project "RIO-128K_ZXspectrum"
         (path "/c309cbb5-591c-4149-a6f5-223f04f1f3af/45e8b7e1-b3fc-453c-b7ce-421d4c8eb212"
-          (reference "#PWR010") (unit 1)
+          (reference "#PWR?") (unit 1)
         )
       )
@@
   (symbol (lib_id "power:GND") (at 160.02 80.01 0) (unit 1)
     (in_bom yes) (on_board yes) (dnp no) (fields_autoplaced)
-    (property "Reference" "#PWR0101" (at 160.02 86.36 0)
+    (property "Reference" "#PWR?" (at 160.02 86.36 0)
       (effects (font (size 1.27 1.27)) hide)
     )
@@
       (project "ZXspectrum_Concept_v2.kicad_pro"
         (path "/532c0392-800e-45cc-8170-6d32f2390e83/8f76c5c7-fe36-4f58-b465-2615c9dcfdfb"
-          (reference "#PWR0101") (unit 1)
+          (reference "#PWR?") (unit 1)
+        )
+      )
+      (project "ZXspectrum_Concept_v2.kicad_pro"
+        (path "/55b3df09-427f-490b-af7e-cf3fd0c70b9f/0d5f1905-044f-4186-8c0e-e74aa689b436"
+          (reference "#PWR019") (unit 1)
         )
       )
       (project "RIO-128K_ZXspectrum"
         (path "/c309cbb5-591c-4149-a6f5-223f04f1f3af/45e8b7e1-b3fc-453c-b7ce-421d4c8eb212"
-          (reference "#PWR011") (unit 1)
+          (reference "#PWR?") (unit 1)
         )
       )
@@
   (symbol (lib_id "Connector:Conn_01x18_Socket") (at 151.13 54.61 0) (mirror y) (unit 1)
     (in_bom yes) (on_board yes) (dnp no) (fields_autoplaced)
-    (property "Reference" "RIO2" (at 151.765 30.48 0)
+    (property "Reference" "RIO?" (at 151.765 30.48 0)
       (effects (font (size 1.27 1.27)))
     )
@@
       (project "ZXspectrum_Concept_v2.kicad_pro"
         (path "/532c0392-800e-45cc-8170-6d32f2390e83/8f76c5c7-fe36-4f58-b465-2615c9dcfdfb"
+          (reference "RIO?") (unit 1)
+        )
+      )
+      (project "ZXspectrum_Concept_v2.kicad_pro"
+        (path "/55b3df09-427f-490b-af7e-cf3fd0c70b9f/0d5f1905-044f-4186-8c0e-e74aa689b436"
           (reference "RIO2") (unit 1)
         )
@@
       (project "RIO-128K_ZXspectrum"
         (path "/c309cbb5-591c-4149-a6f5-223f04f1f3af/45e8b7e1-b3fc-453c-b7ce-421d4c8eb212"
-          (reference "J2") (unit 1)
+          (reference "J?") (unit 1)
         )
       )
@@
   (symbol (lib_id "Connector:Conn_01x24_Socket") (at 90.17 63.5 0) (unit 1)
     (in_bom yes) (on_board yes) (dnp no) (fields_autoplaced)
-    (property "Reference" "RIO1" (at 91.44 64.135 0)
+    (property "Reference" "RIO?" (at 91.44 64.135 0)
       (effects (font (size 1.27 1.27)) (justify left))
     )
@@
       (project "ZXspectrum_Concept_v2.kicad_pro"
         (path "/532c0392-800e-45cc-8170-6d32f2390e83/8f76c5c7-fe36-4f58-b465-2615c9dcfdfb"
+          (reference "RIO?") (unit 1)
+        )
+      )
+      (project "ZXspectrum_Concept_v2.kicad_pro"
+        (path "/55b3df09-427f-490b-af7e-cf3fd0c70b9f/0d5f1905-044f-4186-8c0e-e74aa689b436"
           (reference "RIO1") (unit 1)
         )
@@
       (project "RIO-128K_ZXspectrum"
         (path "/c309cbb5-591c-4149-a6f5-223f04f1f3af/45e8b7e1-b3fc-453c-b7ce-421d4c8eb212"
-          (reference "J1") (unit 1)
-        )
-      )
+          (reference "J?") (unit 1)
+        )
+      )
