File: KiCad7/Z80Bus_Adapters/ZXspectrum_Concept_v2/Impl/SPI-Z80-BUS_ZXspectrum_impl_V2/SPI-Z80-BUS_ZXspectrum_impl_connector.kicad_sch (KiCad schematic)
At the start: 8 parts, among them J1 PinHeader_2.54mm, J5 Z80_CONTROL

Commit message: ThatOldNerds V2 of the concept design.
Parts:
- renumbered J5 to J?, J1 to J?, LOCAL_CONTROL1 to LOCAL_CONTROL?
Connections:
- net !ESP_HARDLOCK renamed ~{ESP_HARDLOCK}
- no-connect marks 0 -> 4
