File: KiCad7/Z80Bus_Adapters/ZXspectrum_Concept_v2/Schem/GLUE_ZXspectrum/RIO CONTROL.kicad_sch (KiCad schematic)
At the start: 12 parts, among them IC1 7404N, IC5 74HC32N, IC6 74HC08N, IC7 74HC32N, U1 74HC244N

Commit message: ThatOldNerds V2 of the concept design.
Parts:
- removed IC1: 7404N, Package_DIP:DIP-14_W7.62mm_Socket, symbol 74xx:74HC04
- removed IC7: 74HC32N, Package_DIP:DIP-14_W7.62mm_Socket, symbol 74xx:74LS32
- added U2: 74HC00, Package_DIP:DIP-14_W7.62mm, symbol 74xx:74HC00
- renumbered D6 to D?, IC5 to IC?, IC6 to IC?, IC7 to IC?, RN1 to RN?, U1 to U?
Connections:
- net PERM_Z80_IORQ is gone; now on net RIO_IOD_DECODE: U?.8 (1A3)
- net RIO_IOD_CONFIG: now also U2.8
- net at IC?.6: now also U2.1, U2.2
- net at IC?.8: now also U2.5
- net RIO_ROM_ACCESS renamed RIO_CONTROL.A16
- new net: U2.3, U2.4
- new net: U2.10, U2.6, U2.9
Other:
- moved on the sheet: IC?A, IC?C, IC?D
