File: KiCad7/Z80Bus_Adapters/ZXspectrum_Concept_v2/Schem/GLUE_ZXspectrum/Z80 BUS CONTROL.kicad_sch (KiCad schematic)
At the start: 7 parts, among them IC11 74HC08N

Commit message: ThatOldNerds V2 of the concept design.
Parts:
- renumbered IC11 to IC?
Connections:
- net ESP_Z80BUS_SAFE_ACCESS renamed Z80_BUS_CONTROL.Z80_ADD_DIR
- net PERM_Z80_IORQ renamed RIO_IOD_DECODE
Other:
- moved on the sheet: IC?A
